Commit message: Adjust gripper position further from end link

File: ur5/src/robotiq/robotiq_2f_140_gripper_visualization/urdf/robotiq_arg2f.xacro (robot description, xacro)
@@ -27,4 +27,5 @@
       		<parent link="${parent}"/>
       		<child link="${prefix}robotiq_arg2f_base_link"/>
+          <origin xyz="0.0 0.0 0.001" rpy="0 0 1.57"/>
     	</joint>
   </xacro:macro>

Commit message: Move away gripper

File: ur5/src/robotiq/robotiq_2f_140_gripper_visualization/urdf/robotiq_arg2f.xacro (robot description, xacro)
@@ -27,5 +27,5 @@
       		<parent link="${parent}"/>
       		<child link="${prefix}robotiq_arg2f_base_link"/>
-          <origin xyz="0.0 0.0 0.001" rpy="0 0 1.57"/>
+          <origin xyz="0.0 0.0 0.005" rpy="0 0 1.57"/>
     	</joint>
   </xacro:macro>

Commit message: Move away gripper from tool0

File: ur5/src/robotiq/robotiq_2f_140_gripper_visualization/urdf/robotiq_arg2f.xacro (robot description, xacro)
@@ -27,5 +27,5 @@
       		<parent link="${parent}"/>
       		<child link="${prefix}robotiq_arg2f_base_link"/>
-          <origin xyz="0.0 0.0 0.005" rpy="0 0 1.57"/>
+          <origin xyz="0.0 0.0 0.006" rpy="0 0 1.57"/>
     	</joint>
   </xacro:macro>

Commit message: New URDF files for the RobotIq 140 2f

File: ur5/src/robotiq/robotiq_2f_140_gripper_visualization/urdf/robotiq_arg2f.xacro (robot description, xacro)
@@ -1,4 +1,5 @@
 <?xml version="1.0"?>
 <robot xmlns:xacro="http://ros.org/wiki/xacro">
+  <!--xacro:include filename="$(find icl_phri_ur5_robotiq_arg140_description)/urdf/robotiq_arg2f_finger_tips.xacro" /-->
   <xacro:macro name="robotiq_arg2f_base_link" params="prefix">
     <link name="${prefix}robotiq_arg2f_base_link">
@@ -11,5 +12,5 @@
         <origin xyz="0 0 0" rpy="0 0 0" />
         <geometry>
-          <mesh filename="package://robotiq_2f_140_gripper_visualization/meshes/robotiq_arg2f_base_link_fine.stl" />
+          <mesh filename="package://icl_ur5_setup_description/meshes/robotiq_arg2f_base_link_fine.stl" />
         </geometry>
         <material name="">
@@ -20,13 +21,8 @@
         <origin xyz="0 0 0" rpy="0 0 ${pi / 2}" />
         <geometry>
-          <mesh filename="package://robotiq_2f_140_gripper_visualization/meshes/robotiq_arg2f_base_link_coarse.stl" />
+          <mesh filename="package://icl_ur5_setup_description/meshes/robotiq_arg2f_base_link_coarse.stl" />
         </geometry>
       </collision>
     </link>
-    <joint name="${prefix}base" type="fixed">
-      		<parent link="${parent}"/>
-      		<child link="${prefix}robotiq_arg2f_base_link"/>
-          <origin xyz="0.0 0.0 0.006" rpy="0 0 1.57"/>
-    	</joint>
   </xacro:macro>
   <xacro:macro name="finger_joints" params="prefix fingerprefix reflect">
@@ -34,4 +30,5 @@
     <xacro:inner_knuckle_joint prefix="${prefix}" fingerprefix="${fingerprefix}" reflect="${reflect}"/>
     <xacro:inner_finger_joint prefix="${prefix}" fingerprefix="${fingerprefix}"/>
+    <xacro:finger_tip_joint prefix="${prefix}" fingerprefix="${fingerprefix}"/>
   </xacro:macro>
   <xacro:macro name="finger_links" params="prefix fingerprefix stroke">
@@ -40,4 +37,5 @@
     <xacro:inner_finger prefix="${prefix}" fingerprefix="${fingerprefix}" stroke="${stroke}"/>
     <xacro:inner_knuckle prefix="${prefix}" fingerprefix="${fingerprefix}" stroke="${stroke}"/>
+    <xacro:finger_tip prefix="${prefix}" fingerprefix="${fingerprefix}" stroke="${stroke}"/>
   </xacro:macro>
 </robot>

File: ur5/src/robotiq/robotiq_2f_140_gripper_visualization/urdf/robotiq_arg2f_140_model.xacro (robot description, xacro)
@@ -1,5 +1,5 @@
 <?xml version="1.0"?>
 <robot name="robotiq_arg2f_140_model" xmlns:xacro="http://ros.org/wiki/xacro">
-  <xacro:include filename="$(find robotiq_2f_140_gripper_visualization)/urdf/robotiq_arg2f_140_model_macro.xacro" />
-  <xacro:robotiq_arg2f_140 prefix="" parent="ee_link"/>
+  <xacro:include filename="$(find icl_ur5_setup_description)/urdf/robotiq_arg2f_140_model_macro.xacro" />
+  <xacro:robotiq_arg2f_140 prefix=""/>
 </robot>

File: ur5/src/robotiq/robotiq_2f_140_gripper_visualization/urdf/robotiq_arg2f_140_model_macro.xacro (robot description, xacro)
@@ -1,5 +1,5 @@
 <?xml version="1.0"?>
 <robot xmlns:xacro="http://ros.org/wiki/xacro">
-  <xacro:include filename="$(find robotiq_2f_140_gripper_visualization)/urdf/robotiq_arg2f_transmission.xacro" />
+  <xacro:include filename="$(find icl_ur5_setup_description)/urdf/robotiq_arg2f_transmission.xacro" />
   <xacro:macro name="outer_knuckle" params="prefix fingerprefix stroke">
     <link name="${prefix}${fingerprefix}_outer_knuckle">
@@ -18,5 +18,5 @@
         <origin xyz="0 0 0" rpy="0 0 0" />
         <geometry>
-          <mesh filename="package://robotiq_2f_140_gripper_visualization/meshes/robotiq_arg2f_${stroke}_outer_knuckle.stl" />
+          <mesh filename="package://icl_ur5_setup_description/meshes/robotiq_arg2f_${stroke}_outer_knuckle.stl" />
         </geometry>
         <material name="">
@@ -27,5 +27,5 @@
         <origin xyz="0 0 0" rpy="0 0 0" />
         <geometry>
-          <mesh filename="package://robotiq_2f_140_gripper_visualization/meshes/robotiq_arg2f_${stroke}_outer_knuckle.stl" />
+          <mesh filename="package://icl_ur5_setup_description/meshes/robotiq_arg2f_${stroke}_outer_knuckle.stl" />
         </geometry>
       </collision>
@@ -48,14 +48,14 @@
         <origin xyz="0 0 0" rpy="0 0 0" />
         <geometry>
-          <mesh filename="package://robotiq_2f_140_gripper_visualization/meshes/robotiq_arg2f_${stroke}_outer_finger.stl" />
-        </geometry>
-        <material name="">
-          <color rgba="0.1 0.1 0.1 1" />
-        </material>
-      </visual>
-      <collision>
-        <origin xyz="0 0 0" rpy="0 0 0" />
-        <geometry>
-          <mesh filename="package://robotiq_2f_140_gripper_visualization/meshes/robotiq_arg2f_${stroke}_outer_finger.stl" />
+          <mesh filename="package://icl_ur5_setup_description/meshes/robotiq_arg2f_${stroke}_outer_finger.stl" />
+        </geometry>
+        <material name="">
+          <color rgba="0.1 0.1 0.1 1" />
+        </material>
+      </visual>
+      <collision>
+        <origin xyz="0 0 0" rpy="0 0 0" />
+        <geometry>
+          <mesh filename="package://icl_ur5_setup_description/meshes/robotiq_arg2f_${stroke}_outer_finger.stl" />
         </geometry>
       </collision>
@@ -78,14 +78,14 @@
         <origin xyz="0 0 0" rpy="0 0 0" />
         <geometry>
-          <mesh filename="package://robotiq_2f_140_gripper_visualization/meshes/robotiq_arg2f_${stroke}_inner_knuckle.stl" />
-        </geometry>
-        <material name="">
-          <color rgba="0.1 0.1 0.1 1" />
-        </material>
-      </visual>
-      <collision>
-        <origin xyz="0 0 0" rpy="0 0 0" />
-        <geometry>
-          <mesh filename="package://robotiq_2f_140_gripper_visualization/meshes/robotiq_arg2f_${stroke}_inner_knuckle.stl" />
+          <mesh filename="package://icl_ur5_setup_description/meshes/robotiq_arg2f_${stroke}_inner_knuckle.stl" />
+        </geometry>
+        <material name="">
+          <color rgba="0.1 0.1 0.1 1" />
+        </material>
+      </visual>
+      <collision>
+        <origin xyz="0 0 0" rpy="0 0 0" />
+        <geometry>
+          <mesh filename="package://icl_ur5_setup_description/meshes/robotiq_arg2f_${stroke}_inner_knuckle.stl" />
         </geometry>
       </collision>
@@ -108,14 +108,14 @@
         <origin xyz="0 0 0" rpy="0 0 0" />
         <geometry>
-          <mesh filename="package://robotiq_2f_140_gripper_visualization/meshes/robotiq_arg2f_${stroke}_inner_finger.stl" />
-        </geometry>
-        <material name="">
-          <color rgba="0.1 0.1 0.1 1" />
-        </material>
-      </visual>
-      <collision>
-        <origin xyz="0 0 0" rpy="0 0 0" />
-        <geometry>
-          <mesh filename="package://robotiq_2f_140_gripper_visualization/meshes/robotiq_arg2f_${stroke}_inner_finger.stl" />
+          <mesh filename="package://icl_ur5_setup_description/meshes/robotiq_arg2f_${stroke}_inner_finger.stl" />
+        </geometry>
+        <material name="">
+          <color rgba="0.1 0.1 0.1 1" />
+        </material>
+      </visual>
+      <collision>
+        <origin xyz="0 0 0" rpy="0 0 0" />
+        <geometry>
+          <mesh filename="package://icl_ur5_setup_description/meshes/robotiq_arg2f_${stroke}_inner_finger.stl" />
         </geometry>
       </collision>
@@ -132,9 +132,10 @@
   <xacro:macro name="inner_knuckle_joint" params="prefix fingerprefix reflect">
     <joint name="${prefix}${fingerprefix}_inner_knuckle_joint" type="revolute">
-      <origin xyz="0 ${reflect * -0.0127} 0.06142" rpy="${pi / 2 + .725} 0 ${(reflect - 1) * pi / 2}" />
+      <origin xyz="0 ${reflect * -0.0127} 0.06142" rpy="${pi / 2 + 0.9} 0 ${(reflect - 1) * pi / 2}" />
       <parent link="${prefix}robotiq_arg2f_base_link" />
       <child link="${prefix}${fingerprefix}_inner_knuckle" />
       <axis xyz="1 0 0" />
-      <limit lower="0" upper="0.8757" velocity="2.0" effort="1000" />
+      <!--<limit lower="0" upper="0.8757" velocity="2.0" effort="1000" /> -->
+	  <limit lower="-3.14159" upper="3.14159" velocity="2.0" effort="1000" />
       <mimic joint="${prefix}finger_joint" multiplier="-1" offset="0" />
     </joint>
@@ -142,19 +143,20 @@
   <xacro:macro name="inner_finger_joint" params="prefix fingerprefix">
     <joint name="${prefix}${fingerprefix}_inner_finger_joint" type="revolute">
-      <origin xyz="0 0.0817554015893473 -0.0282203446692936" rpy="-.725 0 0" />
+      <origin xyz="0 0.0817554015893473 -0.0282203446692936" rpy="-0.9 0 0" />
       <parent link="${prefix}${fingerprefix}_outer_finger" />
       <child link="${prefix}${fingerprefix}_inner_finger" />
       <axis xyz="1 0 0" />
-      <limit lower="0" upper="0.8757" velocity="2.0" effort="1000" />
+      <limit lower="-3.14159" upper="3.14159" velocity="2.0" effort="1000" />
+      <!-- <limit lower="0" upper="0.8757" velocity="2.0" effort="1000" /> -->
       <mimic joint="${prefix}finger_joint" multiplier="1" offset="0" />
     </joint>
   </xacro:macro>
-  <xacro:include filename="$(find robotiq_2f_140_gripper_visualization)/urdf/robotiq_arg2f.xacro" />
   <xacro:macro name="finger_joint" params="prefix">
     <joint name="${prefix}finger_joint" type="revolute">
-      <origin xyz="0 -0.030601 0.054905" rpy="${pi / 2 + .725} 0 0" />
+      <origin xyz="0 -0.030601 0.054905" rpy="${pi / 2 + 0.9} 0 0" />
       <parent link="${prefix}robotiq_arg2f_base_link" />
       <child link="${prefix}left_outer_knuckle" />
       <axis xyz="-1 0 0" />
+      <!-- <limit lower="-3.14159" upper="3.14159" velocity="2.0" effort="1000" /> -->
       <limit lower="0" upper="0.775" velocity="2.0" effort="1000" />
     </joint>
@@ -163,14 +165,56 @@
   <xacro:macro name="right_outer_knuckle_joint" params="prefix">
     <joint name="${prefix}right_outer_knuckle_joint" type="revolute">
-      <origin xyz="0 0.030601 0.054905" rpy="${pi / 2 + .725} 0 ${pi}" />
+      <origin xyz="0 0.030601 0.054905" rpy="${pi / 2 + 0.9} 0 ${pi}" />
       <parent link="${prefix}robotiq_arg2f_base_link" />
       <child link="${prefix}right_outer_knuckle" />
       <axis xyz="1 0 0" />
-      <limit lower="0" upper="0.725" velocity="2.0" effort="1000" />
+      <!-- <limit lower="0" upper="0.725" velocity="2.0" effort="1000" /> -->
+	  <limit lower="-3.14159" upper="3.14159" velocity="2.0" effort="1000" />
     <mimic joint="${prefix}finger_joint" multiplier="-1" offset="0" />
     </joint>
     <xacro:finger_joints prefix="${prefix}" fingerprefix="right" reflect="-1.0"/>
   </xacro:macro>
-  <xacro:macro name="robotiq_arg2f_140" params="prefix parent">
+  <!--finger tip-->
+  <xacro:macro name="finger_tip" params="prefix fingerprefix stroke">
+    <link name="${prefix}${fingerprefix}_finger_tip">
+      <inertial>
+        <origin xyz="0.000299999999999317 0.0160078233491243 -0.0136945669206257" rpy="0 0 0" />
+        <mass value="0.0104003125914103" />
+        <inertia
+            ixx="2.71909453810972E-06"
+            ixy="0.0"
+            ixz="0.0"
+            iyy="7.69100314106116E-07"
+            iyz="0.0"
+            izz="2.30315190420171E-06" />
+      </inertial>
+      <visual>
+        <origin xyz="0 0.02 -0.05" rpy="0 0 0" />
+        <geometry>
+          <mesh filename="package://icl_ur5_setup_description/meshes/robotiq_arg2f_${stroke}_finger_tip.dae" scale="1.0 1.0 1.0"/>
+        </geometry>
+        <material name="">
+          <color rgba="0.1 0.1 0.1 1" />
+        </material>
+      </visual>
+      <collision>
+        <origin xyz="0 0 0" rpy="0 0 0" />
+        <geometry>
+          <mesh filename="package://icl_ur5_setup_description/meshes/robotiq_arg2f_${stroke}_finger_tip.dae" scale="1.0 1.0 1.0"/>
+        </geometry>
+      </collision>
+    </link>
+  </xacro:macro>
+  <xacro:macro name="finger_tip_joint" params="prefix fingerprefix">
+    <joint name="${prefix}${fingerprefix}_finger_tip_joint" type="fixed">
+      <origin xyz="0 0.01821998610742 0.0260018192872234" rpy="0 0 0" />
+      <parent link="${prefix}${fingerprefix}_inner_finger" />
+      <child link="${prefix}${fingerprefix}_finger_tip" />
+      <axis xyz="1 0 0" />
+    </joint>
+  </xacro:macro>
+    <!--Import robotiq desciptions-->
+  <xacro:include filename="$(find icl_ur5_setup_description)/urdf/robotiq_arg2f.xacro" />
+  <xacro:macro name="robotiq_arg2f_140" params="prefix">
     <xacro:robotiq_arg2f_base_link prefix="${prefix}"/>
     <xacro:finger_links prefix="${prefix}" fingerprefix="left" stroke="140"/>

File: ur5/src/robotiq/robotiq_2f_140_gripper_visualization/urdf/robotiq_arg2f_transmission.xacro (robot description, xacro)
@@ -11,73 +11,33 @@
       </actuator>
     </transmission>
-    <gazebo>
-      <!-- loading plugin: mimic joints works in gazebo now-->
-      <plugin filename="libroboticsgroup_gazebo_mimic_joint_plugin.so" name="${prefix}mimic_robotiq_140_4">
-        <joint>${prefix}finger_joint</joint>
-        <mimicJoint>${prefix}right_outer_knuckle_joint</mimicJoint>
-      </plugin>
-      <plugin filename="libroboticsgroup_gazebo_mimic_joint_plugin.so" name="${prefix}mimic_robotiq_140_2">
-        <joint>${prefix}finger_joint</joint>
-        <mimicJoint>${prefix}left_inner_finger_joint</mimicJoint>
-      </plugin>
-      <plugin filename="libroboticsgroup_gazebo_mimic_joint_plugin.so" name="${prefix}mimic_robotiq_140_1">
-        <joint>${prefix}finger_joint</joint>
-        <mimicJoint>${prefix}right_inner_finger_joint</mimicJoint>
-      </plugin>
-      <plugin filename="libroboticsgroup_gazebo_mimic_joint_plugin.so" name="${prefix}mimic_robotiq_140_3">
-        <joint>${prefix}finger_joint</joint>
-        <mimicJoint>${prefix}left_inner_knuckle_joint</mimicJoint>
-      </plugin>
-      <plugin filename="libroboticsgroup_gazebo_mimic_joint_plugin.so" name="${prefix}mimic_robotiq_140_5">
-        <joint>${prefix}finger_joint</joint>
-        <mimicJoint>${prefix}right_inner_knuckle_joint</mimicJoint>
-      </plugin>
-    </gazebo>
-    <!--
-    <transmission name="${prefix}left_inner_finger_joint_trans">
-      <type>transmission_interface/SimpleTransmission</type>
-      <joint name="${prefix}left_inner_finger_joint">
-        <hardwareInterface>EffortJointInterface</hardwareInterface>
-      </joint>
-      <actuator name="${prefix}finger_joint_motor">
-        <mechanicalReduction>1</mechanicalReduction>
-      </actuator>
-    </transmission>
-    <transmission name="${prefix}left_inner_knuckle_joint_trans">
-      <type>transmission_interface/SimpleTransmission</type>
-      <joint name="${prefix}left_inner_knuckle_joint">
-        <hardwareInterface>EffortJointInterface</hardwareInterface>
-      </joint>
-      <actuator name="${prefix}finger_joint_motor">
-        <mechanicalReduction>1</mechanicalReduction>
-      </actuator>
-    </transmission>
-    <transmission name="${prefix}right_inner_knuckle_joint_trans">
-      <type>transmission_interface/SimpleTransmission</type>
-      <joint name="${prefix}right_inner_knuckle_joint">
-        <hardwareInterface>EffortJointInterface</hardwareInterface>
-      </joint>
-      <actuator name="${prefix}finger_joint_motor">
-        <mechanicalReduction>1</mechanicalReduction>
-      </actuator>
-    </transmission>
-    <transmission name="${prefix}right_outer_knuckle_joint_trans">
-      <type>transmission_interface/SimpleTransmission</type>
-      <joint name="${prefix}right_outer_knuckle_joint">
-        <hardwareInterface>EffortJointInterface</hardwareInterface>
-      </joint>
-      <actuator name="${prefix}finger_joint_motor">
-        <mechanicalReduction>1</mechanicalReduction>
-      </actuator>
-    </transmission>
-    <transmission name="${prefix}right_inner_finger_joint_trans">
-      <type>transmission_interface/SimpleTransmission</type>
-      <joint name="${prefix}right_inner_finger_joint">
-        <hardwareInterface>EffortJointInterface</hardwareInterface>
-      </joint>
-      <actuator name="${prefix}finger_joint_motor">
-        <mechanicalReduction>1</mechanicalReduction>
-      </actuator>
-    </transmission> -->
+	    <gazebo>
+             <!-- loading plugin: mimic joints works in gazebo now-->
+             <plugin filename="libroboticsgroup_gazebo_mimic_joint_plugin.so" name="${prefix}mimic_robotiq_140_4">
+                <joint>${prefix}finger_joint</joint>
+                <mimicJoint>${prefix}right_outer_knuckle_joint</mimicJoint>
+                <multiplier>-1.0</multiplier>
+            </plugin>
+            <plugin filename="libroboticsgroup_gazebo_mimic_joint_plugin.so" name="${prefix}mimic_robotiq_140_2">
+                <joint>${prefix}finger_joint</joint>
+                <mimicJoint>${prefix}left_inner_finger_joint</mimicJoint>
+                <multiplier>1.0</multiplier>
+                <!--<offset>0.0</offset>-->
+            </plugin>
+            <plugin filename="libroboticsgroup_gazebo_mimic_joint_plugin.so" name="${prefix}mimic_robotiq_140_1">
+                <joint>${prefix}finger_joint</joint>
+                <mimicJoint>${prefix}right_inner_finger_joint</mimicJoint>
+                <multiplier>1.0</multiplier>
+            </plugin>
+            <plugin filename="libroboticsgroup_gazebo_mimic_joint_plugin.so" name="${prefix}mimic_robotiq_140_3">
+                <joint>${prefix}finger_joint</joint>
+                <mimicJoint>${prefix}left_inner_knuckle_joint</mimicJoint>
+                <multiplier>-1.0</multiplier>
+            </plugin>
+            <plugin filename="libroboticsgroup_gazebo_mimic_joint_plugin.so" name="${prefix}mimic_robotiq_140_5">
+                <joint>${prefix}finger_joint</joint>
+                <mimicJoint>${prefix}right_inner_knuckle_joint</mimicJoint>
+                <multiplier>-1.0</multiplier>
+            </plugin>
+        </gazebo>
   </xacro:macro>
 </robot>

Commit message: Change directory for the original RobotIq packages

File: ur5/src/robotiq/robotiq_2f_140_gripper_visualization/urdf/robotiq_arg2f.xacro (robot description, xacro)
@@ -12,5 +12,5 @@
         <origin xyz="0 0 0" rpy="0 0 0" />
         <geometry>
-          <mesh filename="package://icl_ur5_setup_description/meshes/robotiq_arg2f_base_link_fine.stl" />
+          <mesh filename="package://robotiq_2f_140_gripper_visualization/meshes/robotiq_arg2f_base_link_fine.stl" />
         </geometry>
         <material name="">
@@ -21,5 +21,5 @@
         <origin xyz="0 0 0" rpy="0 0 ${pi / 2}" />
         <geometry>
-          <mesh filename="package://icl_ur5_setup_description/meshes/robotiq_arg2f_base_link_coarse.stl" />
+          <mesh filename="package://robotiq_2f_140_gripper_visualization/meshes/robotiq_arg2f_base_link_coarse.stl" />
         </geometry>
       </collision>
