Commit message: Change directory for the original RobotIq packages

File: ur5/src/robotiq/robotiq_2f_140_gripper_visualization/urdf/robotiq_arg2f_140_model_macro.xacro (robot description, xacro)
@@ -1,5 +1,5 @@
 <?xml version="1.0"?>
 <robot xmlns:xacro="http://ros.org/wiki/xacro">
-  <xacro:include filename="$(find icl_ur5_setup_description)/urdf/robotiq_arg2f_transmission.xacro" />
+  <xacro:include filename="$(find robotiq_2f_140_gripper_visualization)/urdf/robotiq_arg2f_transmission.xacro" />
   <xacro:macro name="outer_knuckle" params="prefix fingerprefix stroke">
     <link name="${prefix}${fingerprefix}_outer_knuckle">
@@ -18,5 +18,5 @@
         <origin xyz="0 0 0" rpy="0 0 0" />
         <geometry>
-          <mesh filename="package://icl_ur5_setup_description/meshes/robotiq_arg2f_${stroke}_outer_knuckle.stl" />
+          <mesh filename="package://robotiq_2f_140_gripper_visualization/meshes/robotiq_arg2f_${stroke}_outer_knuckle.stl" />
         </geometry>
         <material name="">
@@ -27,5 +27,5 @@
         <origin xyz="0 0 0" rpy="0 0 0" />
         <geometry>
-          <mesh filename="package://icl_ur5_setup_description/meshes/robotiq_arg2f_${stroke}_outer_knuckle.stl" />
+          <mesh filename="package://robotiq_2f_140_gripper_visualization/meshes/robotiq_arg2f_${stroke}_outer_knuckle.stl" />
         </geometry>
       </collision>
@@ -48,14 +48,14 @@
         <origin xyz="0 0 0" rpy="0 0 0" />
         <geometry>
-          <mesh filename="package://icl_ur5_setup_description/meshes/robotiq_arg2f_${stroke}_outer_finger.stl" />
-        </geometry>
-        <material name="">
-          <color rgba="0.1 0.1 0.1 1" />
-        </material>
-      </visual>
-      <collision>
-        <origin xyz="0 0 0" rpy="0 0 0" />
-        <geometry>
-          <mesh filename="package://icl_ur5_setup_description/meshes/robotiq_arg2f_${stroke}_outer_finger.stl" />
+          <mesh filename="package://robotiq_2f_140_gripper_visualization/meshes/robotiq_arg2f_${stroke}_outer_finger.stl" />
+        </geometry>
+        <material name="">
+          <color rgba="0.1 0.1 0.1 1" />
+        </material>
+      </visual>
+      <collision>
+        <origin xyz="0 0 0" rpy="0 0 0" />
+        <geometry>
+          <mesh filename="package://robotiq_2f_140_gripper_visualization/meshes/robotiq_arg2f_${stroke}_outer_finger.stl" />
         </geometry>
       </collision>
@@ -78,14 +78,14 @@
         <origin xyz="0 0 0" rpy="0 0 0" />
         <geometry>
-          <mesh filename="package://icl_ur5_setup_description/meshes/robotiq_arg2f_${stroke}_inner_knuckle.stl" />
-        </geometry>
-        <material name="">
-          <color rgba="0.1 0.1 0.1 1" />
-        </material>
-      </visual>
-      <collision>
-        <origin xyz="0 0 0" rpy="0 0 0" />
-        <geometry>
-          <mesh filename="package://icl_ur5_setup_description/meshes/robotiq_arg2f_${stroke}_inner_knuckle.stl" />
+          <mesh filename="package://robotiq_2f_140_gripper_visualization/meshes/robotiq_arg2f_${stroke}_inner_knuckle.stl" />
+        </geometry>
+        <material name="">
+          <color rgba="0.1 0.1 0.1 1" />
+        </material>
+      </visual>
+      <collision>
+        <origin xyz="0 0 0" rpy="0 0 0" />
+        <geometry>
+          <mesh filename="package://robotiq_2f_140_gripper_visualization/meshes/robotiq_arg2f_${stroke}_inner_knuckle.stl" />
         </geometry>
       </collision>
@@ -108,14 +108,14 @@
         <origin xyz="0 0 0" rpy="0 0 0" />
         <geometry>
-          <mesh filename="package://icl_ur5_setup_description/meshes/robotiq_arg2f_${stroke}_inner_finger.stl" />
-        </geometry>
-        <material name="">
-          <color rgba="0.1 0.1 0.1 1" />
-        </material>
-      </visual>
-      <collision>
-        <origin xyz="0 0 0" rpy="0 0 0" />
-        <geometry>
-          <mesh filename="package://icl_ur5_setup_description/meshes/robotiq_arg2f_${stroke}_inner_finger.stl" />
+          <mesh filename="package://robotiq_2f_140_gripper_visualization/meshes/robotiq_arg2f_${stroke}_inner_finger.stl" />
+        </geometry>
+        <material name="">
+          <color rgba="0.1 0.1 0.1 1" />
+        </material>
+      </visual>
+      <collision>
+        <origin xyz="0 0 0" rpy="0 0 0" />
+        <geometry>
+          <mesh filename="package://robotiq_2f_140_gripper_visualization/meshes/robotiq_arg2f_${stroke}_inner_finger.stl" />
         </geometry>
       </collision>
@@ -192,14 +192,14 @@
         <origin xyz="0 0.02 -0.05" rpy="0 0 0" />
         <geometry>
-          <mesh filename="package://icl_ur5_setup_description/meshes/robotiq_arg2f_${stroke}_finger_tip.dae" scale="1.0 1.0 1.0"/>
-        </geometry>
-        <material name="">
-          <color rgba="0.1 0.1 0.1 1" />
-        </material>
-      </visual>
-      <collision>
-        <origin xyz="0 0 0" rpy="0 0 0" />
-        <geometry>
-          <mesh filename="package://icl_ur5_setup_description/meshes/robotiq_arg2f_${stroke}_finger_tip.dae" scale="1.0 1.0 1.0"/>
+          <mesh filename="package://robotiq_2f_140_gripper_visualization/meshes/robotiq_arg2f_${stroke}_finger_tip.dae" scale="1.0 1.0 1.0"/>
+        </geometry>
+        <material name="">
+          <color rgba="0.1 0.1 0.1 1" />
+        </material>
+      </visual>
+      <collision>
+        <origin xyz="0 0 0" rpy="0 0 0" />
+        <geometry>
+          <mesh filename="package://robotiq_2f_140_gripper_visualization/meshes/robotiq_arg2f_${stroke}_finger_tip.dae" scale="1.0 1.0 1.0"/>
         </geometry>
       </collision>
@@ -215,5 +215,5 @@
   </xacro:macro>
     <!--Import robotiq desciptions-->
-  <xacro:include filename="$(find icl_ur5_setup_description)/urdf/robotiq_arg2f.xacro" />
+  <xacro:include filename="$(find robotiq_2f_140_gripper_visualization)/urdf/robotiq_arg2f.xacro" />
   <xacro:macro name="robotiq_arg2f_140" params="prefix">
     <xacro:robotiq_arg2f_base_link prefix="${prefix}"/>
