Commit message: Add camera to robot.urdf and gripper parent link set to tool0

File: ur5/src/universal_robot/ur_description/urdf/ur5_robot.urdf.xacro (robot description, xacro)
@@ -11,4 +11,9 @@
     transmission_hw_interface="$(arg transmission_hw_interface)"
   />
+  <xacro:include filename="$(find ur_description)/urdf/camera/camera.urdf.xacro"/>
+  <xacro:camera_v0 parent="base_link">
+	     <origin xyz="1.0 -1.0 0.15" rpy="0 -0.2 2.39"/>
+  </xacro:camera_v0>
+  <xacro:camera_gazebo_v0 />
   <link name="world" />
   <joint name="world_joint" type="fixed">
@@ -18,4 +23,4 @@
   </joint>
    <xacro:include filename="$(find robotiq_2f_140_gripper_visualization)/urdf/robotiq_arg2f_140_model_macro.xacro" />
-  <xacro:robotiq_arg2f_140 prefix="" parent="ee_link"/>
+  <xacro:robotiq_arg2f_140 prefix="" parent="tool0"/>
 </robot>

Commit message: Import gripper to UR5 URDF

File: ur5/src/universal_robot/ur_description/urdf/ur5_robot.urdf.xacro (robot description, xacro)
@@ -5,4 +5,5 @@
   <!-- common stuff -->
   <xacro:include filename="$(find ur_description)/urdf/common.gazebo.xacro" />
+  <xacro:include filename="$(find robotiq_2f_140_gripper_visualization)/urdf/robotiq_arg2f_140_model_macro.xacro" />
   <!-- ur5 -->
   <xacro:include filename="$(find ur_description)/urdf/ur5.urdf.xacro" />
@@ -24,3 +25,10 @@
   <!--xacro:include filename="$(find robotiq_2f_140_gripper_visualization)/urdf/robotiq_arg2f_140_model_macro.xacro" />
   <xacro:robotiq_arg2f_140 prefix="" parent="tool0"/-->
+   <!-- gripper -->
+    <xacro:robotiq_arg2f_140 prefix="" />
+    <joint name="ur5_ee_link_gripper_base" type="fixed">
+      <parent link= "tool0" />
+      <child link = "robotiq_arg2f_base_link" />
+      <origin xyz=" 0.0 0.0 0.0" rpy="0.0 0.0 ${pi/2}" />
+    </joint>
 </robot>

Commit message: Update ur5_robot.urdf.xacro

File: ur5/src/universal_robot/ur_description/urdf/ur5_robot.urdf.xacro (robot description, xacro)
@@ -32,3 +32,9 @@
       <origin xyz=" 0.0 0.0 0.0" rpy="0.0 0.0 ${pi/2}" />
     </joint>
+    <link name="tool" />
+    <joint name="tool_tip" type="fixed">
+      <parent link= "ee_link" />
+      <child link = "tool" />
+      <origin xyz=" 0.00 0.0 0.2" rpy="0.0 0.0 0.0" />
+    </joint>
 </robot>
