Commit message: Purge repository and add default robotiq packages

File: ur5/src/universal_robot/ur_e_description/urdf/ur.transmission.xacro (robot description, xacro)
@@ -5,5 +5,5 @@
       <type>transmission_interface/SimpleTransmission</type>
       <joint name="${prefix}shoulder_pan_joint">
-        <hardwareInterface>hardware_interface/PositionJointInterface</hardwareInterface>
+        <hardwareInterface>EffortJointInterface</hardwareInterface>
       </joint>
       <actuator name="${prefix}shoulder_pan_motor">
@@ -14,5 +14,5 @@
       <type>transmission_interface/SimpleTransmission</type>
       <joint name="${prefix}shoulder_lift_joint">
-        <hardwareInterface>hardware_interface/PositionJointInterface</hardwareInterface>
+        <hardwareInterface>EffortJointInterface</hardwareInterface>
       </joint>
       <actuator name="${prefix}shoulder_lift_motor">
@@ -23,5 +23,5 @@
       <type>transmission_interface/SimpleTransmission</type>
       <joint name="${prefix}elbow_joint">
-        <hardwareInterface>hardware_interface/PositionJointInterface</hardwareInterface>
+        <hardwareInterface>EffortJointInterface</hardwareInterface>
       </joint>
       <actuator name="${prefix}elbow_motor">
@@ -32,5 +32,5 @@
       <type>transmission_interface/SimpleTransmission</type>
       <joint name="${prefix}wrist_1_joint">
-        <hardwareInterface>hardware_interface/PositionJointInterface</hardwareInterface>
+        <hardwareInterface>EffortJointInterface</hardwareInterface>
       </joint>
       <actuator name="${prefix}wrist_1_motor">
@@ -41,5 +41,5 @@
       <type>transmission_interface/SimpleTransmission</type>
       <joint name="${prefix}wrist_2_joint">
-        <hardwareInterface>hardware_interface/PositionJointInterface</hardwareInterface>
+        <hardwareInterface>EffortJointInterface</hardwareInterface>
       </joint>
       <actuator name="${prefix}wrist_2_motor">
@@ -50,5 +50,5 @@
       <type>transmission_interface/SimpleTransmission</type>
       <joint name="${prefix}wrist_3_joint">
-        <hardwareInterface>hardware_interface/PositionJointInterface</hardwareInterface>
+        <hardwareInterface>EffortJointInterface</hardwareInterface>
       </joint>
       <actuator name="${prefix}wrist_3_motor">

File: ur5/src/universal_robot/ur_e_description/urdf/ur5e_robot.urdf.xacro (robot description, xacro)
@@ -4,4 +4,16 @@
   <!-- common stuff -->
   <xacro:include filename="$(find ur_e_description)/urdf/common.gazebo.xacro" />
+  <xacro:include filename="$(find robotiq_2f_140_gripper_visualization)/urdf/robotiq_arg2f_140_model_macro.xacro" />
+  <xacro:include filename="$(find robotiq_3f_gripper_visualization)/cfg/robotiq-3f-gripper_articulated_macro.xacro" />
+  <xacro:include filename="$(find ur_e_description)/urdf/camera/camera.urdf.xacro"/>
+  <xacro:include filename="$(find ur_e_description)/urdf/camera2/camera.urdf.xacro"/>
+  <xacro:camera_v0 parent="base_link">
+	     <origin xyz="1.5 0.0 0.5" rpy="0 0.0 3.1415"/>
+  </xacro:camera_v0>
+  <xacro:camera_gazebo_v0 />
+  <xacro:camera_v1 parent="base_link">
+	     <origin xyz="0.0 1.5 0.5" rpy="0 0.0 -1.57"/>
+  </xacro:camera_v1>
+  <xacro:camera_gazebo_v1 />
   <!-- ur5e -->
   <xacro:include filename="$(find ur_e_description)/urdf/ur5e.urdf.xacro" />
@@ -14,3 +26,21 @@
     <origin xyz="0.0 0.0 0.0" rpy="0.0 0.0 0.0" />
   </joint>
+ <xacro:robotiq_arg2f_140 prefix="" />
+    <joint name="ur5_ee_link_gripper_base" type="fixed">
+      <parent link= "tool0" />
+      <child link = "robotiq_arg2f_base_link" />
+      <origin xyz=" 0.0 0.0 0.0" rpy="0.0 0.0 ${pi/2}" />
+    </joint>
+    <link name="tool" />
+    <joint name="tool_tip" type="fixed">
+      <parent link= "ee_link" />
+      <child link = "tool" />
+      <origin xyz=" 0.00 0.0 0.2" rpy="0.0 0.0 0.0" />
+    </joint>
+  <!--xacro:robotiq-3f-gripper_articulated prefix="gripper_"/>
+    <joint name="base_gripper" type="fixed">
+      <parent link= "tool0" />
+      <child link = "gripper_palm" />
+      <origin xyz=" 0.0 0.0 0.1" rpy="${pi/2} 0.0 0.0" />
+    </joint-->
 </robot>
