Commit message: Robotiq 3f from summer
Change the original robotiq modelling for the one from summer repository. It adds the motor transmissions and some dynamics and friction values

File: src/robotiq/robotiq_3f_gripper_visualization/cfg/robotiq-3f-gripper_articulated_macro.xacro (robot description, xacro)
@@ -6,6 +6,8 @@
 -->
 <robot xmlns:xacro="http://ros.org/wiki/xacro">
+        <xacro:property name="s1" value="0.85" />
+        <xacro:property name="e1" value="40" />
         <xacro:include filename="$(find robotiq_3f_gripper_visualization)/cfg/robotiq-3f-gripper_finger_articulated_macro.xacro" />
-        <xacro:macro name="robotiq-3f-gripper_articulated" params="prefix">
+        <xacro:macro name="robotiq-3f-gripper_articulated" params="prefix *origin reflect parent">
         <xacro:robotiq-3f-gripper_finger_articulated prefix="${prefix}finger_1_"/>
         <xacro:robotiq-3f-gripper_finger_articulated prefix="${prefix}finger_2_"/>
@@ -15,5 +17,5 @@
 			<visual>
 				<geometry>
-                                        <mesh filename="package://robotiq_3f_gripper_visualization/meshes/robotiq-3f-gripper_articulated/visual/palm.dae" />
+                                        <mesh filename="package://robotiq_3f_gripper_visualization/meshes/robotiq-3f-gripper_articulated/visual/palm.STL" />
 				</geometry>
 				<material name="gray">
@@ -30,5 +32,8 @@
 			</collision>
 		</link>
-		<link name="${prefix}tool0"/>
+	    <gazebo reference="${prefix}palm">
+      		<mu1>1.1</mu1>
+      		<mu2>1.1</mu2>
+    	</gazebo>
         <inertial>
             <origin xyz="0 0 0" rpy="0 0 0"/>
@@ -43,5 +48,5 @@
 			<axis xyz="0 1 0"/>
 			<origin xyz="-0.0455 0.0214 0.036" rpy="0 3.1416 -1.57"/>
-			<limit lower="-0.1784" upper="0.192" effort="100" velocity="100"/>
+                        <limit lower="-0.1784" upper="0.192" effort="100" velocity="${s1}"/>
 		</joint>
 		<joint name="${prefix}palm_finger_2_joint" type="revolute">
@@ -50,5 +55,5 @@
 			<axis xyz="0 1 0"/>
 			<origin xyz="-0.0455 0.0214 -0.036" rpy="0 3.1416 -1.57"/>
-			<limit lower="-0.192" upper="0.1784" effort="100" velocity="100"/>
+                        <limit lower="-0.192" upper="0.1784" effort="100" velocity="${s1}"/>
 		</joint>
 		<joint name="${prefix}palm_finger_middle_joint" type="fixed">
@@ -58,9 +63,22 @@
 			<origin xyz="0.0455 0.0214 0" rpy="0 0 1.57"/>
 		</joint>
-		<joint name="${prefix}palm_tool0" type="fixed">
-			<parent link="${prefix}palm"/>
-			<child link="${prefix}tool0"/>
-			<origin xyz="0.0 0.0875 0.0" rpy="0 0 1.5707"/>
-		</joint>
+    <transmission name="${prefix}palm_finger_1_trans">
+      <type>transmission_interface/SimpleTransmission</type>
+      <joint name="${prefix}palm_finger_1_joint">
+        <hardwareInterface>hardware_interface/EffortJointInterface</hardwareInterface>
+      </joint>
+      <actuator name="${prefix}palm_finger_1_motor">
+        <mechanicalReduction>1</mechanicalReduction>
+      </actuator>
+    </transmission>
+    <transmission name="${prefix}palm_finger_2_trans">
+      <type>transmission_interface/SimpleTransmission</type>
+      <joint name="${prefix}palm_finger_2_joint">
+        <hardwareInterface>hardware_interface/EffortJointInterface</hardwareInterface>
+      </joint>
+      <actuator name="${prefix}palm_finger_2_motor">
+        <mechanicalReduction>1</mechanicalReduction>
+      </actuator>
+    </transmission>
 		<!-- end of joint list -->
 	</xacro:macro>

File: src/robotiq/robotiq_3f_gripper_visualization/cfg/robotiq-3f-gripper_finger_articulated_macro.xacro (robot description, xacro)
@@ -6,5 +6,8 @@
 -->
 <robot xmlns:xacro="http://ros.org/wiki/xacro">
+        <xacro:property name="s1" value="0.88" />
+        <xacro:property name="e1" value="100" />
         <xacro:macro name="robotiq-3f-gripper_finger_articulated" params="prefix">
+		<xacro:include filename="$(find robotiq_3f_gripper_visualization)/cfg/robotiq.transmission.xacro" />
 		<!-- link list -->
 		<link name="${prefix}link_0">
@@ -12,5 +15,5 @@
 				<origin xyz="0.020 0 0" rpy="0 0 0"/>
 				<geometry>
-                                        <mesh filename="package://robotiq_3f_gripper_visualization/meshes/robotiq-3f-gripper_articulated/visual/link_0.dae" />
+                                        <mesh filename="package://robotiq_3f_gripper_visualization/meshes/robotiq-3f-gripper_articulated/visual/link_0.STL" />
 				</geometry>
 				<material name="gray">
@@ -33,9 +36,13 @@
             </inertial>
 		</link>
+		<gazebo reference="${prefix}link_0">
+      		<mu1>1.1</mu1>
+      		<mu2>1.1</mu2>
+    	</gazebo>
 		<link name="${prefix}link_1">
 			<visual>
 				<origin xyz="0.050 -.028 0" rpy="0 0 -0.52"/>
 				<geometry>
-                                        <mesh filename="package://robotiq_3f_gripper_visualization/meshes/robotiq-3f-gripper_articulated/visual/link_1.dae" />
+                                        <mesh filename="package://robotiq_3f_gripper_visualization/meshes/robotiq-3f-gripper_articulated/visual/link_1.STL" />
 				</geometry>
 				<material name="gray"/>
@@ -54,4 +61,8 @@
             </inertial>
 		</link>
+		<gazebo reference="${prefix}link_1">
+      		<mu1>1.1</mu1>
+      		<mu2>1.1</mu2>
+    	</gazebo>
 		<link name="${prefix}link_2">
 			<!--
@@ -63,5 +74,5 @@
 				<origin xyz="0.039 0 0.0075" rpy="0 0 0"/>
 				<geometry>
-                                        <mesh filename="package://robotiq_3f_gripper_visualization/meshes/robotiq-3f-gripper_articulated/visual/link_2.dae" />
+                                        <mesh filename="package://robotiq_3f_gripper_visualization/meshes/robotiq-3f-gripper_articulated/visual/link_2.STL" />
 				</geometry>
 				<material name="gray"/>
@@ -80,9 +91,13 @@
             </inertial>
 		</link>
+		<gazebo reference="${prefix}link_2">
+      		<mu1>1.1</mu1>
+      		<mu2>1.1</mu2>
+    	</gazebo>
 		<link name="${prefix}link_3">
 			<visual>
 				<origin xyz="0 0 0" rpy="0 0 0.52"/>
 				<geometry>
-                                        <mesh filename="package://robotiq_3f_gripper_visualization/meshes/robotiq-3f-gripper_articulated/visual/link_3.dae" />
+                                        <mesh filename="package://robotiq_3f_gripper_visualization/meshes/robotiq-3f-gripper_articulated/visual/link_3.STL" />
 				</geometry>
 				<material name="gray"/>
@@ -101,6 +116,11 @@
             </inertial>
 		</link>
+		<gazebo reference="${prefix}link_3">
+      		<mu1>1.1</mu1>
+      		<mu2>1.1</mu2>
+    	</gazebo>
 		<!-- end of link list -->
 		<!-- joint list -->
+		<xacro:robotiq_transmission prefix="${prefix}" />
 		<joint name="${prefix}joint_1" type="revolute">
 			<parent link="${prefix}link_0"/>
@@ -108,5 +128,5 @@
 			<axis xyz="0 0 1"/>
 			<origin xyz="0.020 0 0" rpy="0 0 0"/>
-			<limit lower="0.0495" upper="1.2218" effort="100" velocity="100"/>
+                        <limit lower="0.0495" upper="1.2218" effort="${e1}" velocity="${s1}"/>
 		</joint>
 		<joint name="${prefix}joint_2" type="revolute">
@@ -115,5 +135,5 @@
 			<axis xyz="0 0 1"/>
 			<origin xyz="0.050 -.028 0" rpy="0 0 -0.52"/>
-			<limit lower="0.0" upper="1.5708" effort="100" velocity="100"/>
+                        <limit lower="0.0" upper="1.5708" effort="${e1}" velocity="${s1}"/>
 		</joint>
 		<joint name="${prefix}joint_3" type="revolute">
@@ -122,5 +142,5 @@
 			<axis xyz="0 0 1"/>
 			<origin xyz="0.039 0 0" rpy="0 0 0"/>
-			<limit lower="-1.2217" upper="-0.0523" effort="100" velocity="100"/>
+                        <limit lower="-1.2217" upper="-0.074532925" effort="${e1}" velocity="${s1}"/>
 		</joint>
 		<!-- end of joint list -->

Commit message: Original robotiq 3f gripper files with transmissions

File: src/robotiq/robotiq_3f_gripper_visualization/cfg/robotiq-3f-gripper_articulated_macro.xacro (robot description, xacro)
@@ -6,8 +6,6 @@
 -->
 <robot xmlns:xacro="http://ros.org/wiki/xacro">
-        <xacro:property name="s1" value="0.85" />
-        <xacro:property name="e1" value="40" />
         <xacro:include filename="$(find robotiq_3f_gripper_visualization)/cfg/robotiq-3f-gripper_finger_articulated_macro.xacro" />
-        <xacro:macro name="robotiq-3f-gripper_articulated" params="prefix *origin reflect parent">
+        <xacro:macro name="robotiq-3f-gripper_articulated" params="prefix">
         <xacro:robotiq-3f-gripper_finger_articulated prefix="${prefix}finger_1_"/>
         <xacro:robotiq-3f-gripper_finger_articulated prefix="${prefix}finger_2_"/>
@@ -17,5 +15,5 @@
 			<visual>
 				<geometry>
-                                        <mesh filename="package://robotiq_3f_gripper_visualization/meshes/robotiq-3f-gripper_articulated/visual/palm.STL" />
+                                        <mesh filename="package://robotiq_3f_gripper_visualization/meshes/robotiq-3f-gripper_articulated/visual/palm.dae" />
 				</geometry>
 				<material name="gray">
@@ -32,8 +30,5 @@
 			</collision>
 		</link>
-	    <gazebo reference="${prefix}palm">
-      		<mu1>1.1</mu1>
-      		<mu2>1.1</mu2>
-    	</gazebo>
+		<link name="${prefix}tool0"/>
         <inertial>
             <origin xyz="0 0 0" rpy="0 0 0"/>
@@ -48,5 +43,5 @@
 			<axis xyz="0 1 0"/>
 			<origin xyz="-0.0455 0.0214 0.036" rpy="0 3.1416 -1.57"/>
-                        <limit lower="-0.1784" upper="0.192" effort="100" velocity="${s1}"/>
+			<limit lower="-0.1784" upper="0.192" effort="100" velocity="100"/>
 		</joint>
 		<joint name="${prefix}palm_finger_2_joint" type="revolute">
@@ -55,5 +50,5 @@
 			<axis xyz="0 1 0"/>
 			<origin xyz="-0.0455 0.0214 -0.036" rpy="0 3.1416 -1.57"/>
-                        <limit lower="-0.192" upper="0.1784" effort="100" velocity="${s1}"/>
+			<limit lower="-0.192" upper="0.1784" effort="100" velocity="100"/>
 		</joint>
 		<joint name="${prefix}palm_finger_middle_joint" type="fixed">
@@ -63,23 +58,29 @@
 			<origin xyz="0.0455 0.0214 0" rpy="0 0 1.57"/>
 		</joint>
-    <transmission name="${prefix}palm_finger_1_trans">
-      <type>transmission_interface/SimpleTransmission</type>
-      <joint name="${prefix}palm_finger_1_joint">
-        <hardwareInterface>hardware_interface/EffortJointInterface</hardwareInterface>
-      </joint>
-      <actuator name="${prefix}palm_finger_1_motor">
-        <mechanicalReduction>1</mechanicalReduction>
-      </actuator>
-    </transmission>
-    <transmission name="${prefix}palm_finger_2_trans">
-      <type>transmission_interface/SimpleTransmission</type>
-      <joint name="${prefix}palm_finger_2_joint">
-        <hardwareInterface>hardware_interface/EffortJointInterface</hardwareInterface>
-      </joint>
-      <actuator name="${prefix}palm_finger_2_motor">
-        <mechanicalReduction>1</mechanicalReduction>
-      </actuator>
-    </transmission>
+		<joint name="${prefix}palm_tool0" type="fixed">
+			<parent link="${prefix}palm"/>
+			<child link="${prefix}tool0"/>
+			<origin xyz="0.0 0.0875 0.0" rpy="0 0 1.5707"/>
+		</joint>
 		<!-- end of joint list -->
-	</xacro:macro>
+		<!-- Palm transmissions -->
+		<transmission name="${prefix}palm_finger_1_trans">
+			<type>transmission_interface/SimpleTransmission</type>
+			<joint name="${prefix}palm_finger_1_joint">
+				<hardwareInterface>hardware_interface/EffortJointInterface</hardwareInterface>
+			</joint>
+			<actuator name="${prefix}palm_finger_1_motor">
+				<mechanicalReduction>1</mechanicalReduction>
+			</actuator>
+		</transmission>
+		<transmission name="${prefix}palm_finger_2_trans">
+			<type>transmission_interface/SimpleTransmission</type>
+			<joint name="${prefix}palm_finger_2_joint">
+				<hardwareInterface>hardware_interface/EffortJointInterface</hardwareInterface>
+			</joint>
+			<actuator name="${prefix}palm_finger_2_motor">
+				<mechanicalReduction>1</mechanicalReduction>
+			</actuator>
+			</transmission>
+		</xacro:macro>
 </robot>

File: src/robotiq/robotiq_3f_gripper_visualization/cfg/robotiq-3f-gripper_finger_articulated_macro.xacro (robot description, xacro)
@@ -6,6 +6,4 @@
 -->
 <robot xmlns:xacro="http://ros.org/wiki/xacro">
-        <xacro:property name="s1" value="0.88" />
-        <xacro:property name="e1" value="100" />
         <xacro:macro name="robotiq-3f-gripper_finger_articulated" params="prefix">
 		<xacro:include filename="$(find robotiq_3f_gripper_visualization)/cfg/robotiq.transmission.xacro" />
@@ -15,5 +13,5 @@
 				<origin xyz="0.020 0 0" rpy="0 0 0"/>
 				<geometry>
-                                        <mesh filename="package://robotiq_3f_gripper_visualization/meshes/robotiq-3f-gripper_articulated/visual/link_0.STL" />
+                                        <mesh filename="package://robotiq_3f_gripper_visualization/meshes/robotiq-3f-gripper_articulated/visual/link_0.dae" />
 				</geometry>
 				<material name="gray">
@@ -36,13 +34,9 @@
             </inertial>
 		</link>
-		<gazebo reference="${prefix}link_0">
-      		<mu1>1.1</mu1>
-      		<mu2>1.1</mu2>
-    	</gazebo>
 		<link name="${prefix}link_1">
 			<visual>
 				<origin xyz="0.050 -.028 0" rpy="0 0 -0.52"/>
 				<geometry>
-                                        <mesh filename="package://robotiq_3f_gripper_visualization/meshes/robotiq-3f-gripper_articulated/visual/link_1.STL" />
+                                        <mesh filename="package://robotiq_3f_gripper_visualization/meshes/robotiq-3f-gripper_articulated/visual/link_1.dae" />
 				</geometry>
 				<material name="gray"/>
@@ -61,8 +55,4 @@
             </inertial>
 		</link>
-		<gazebo reference="${prefix}link_1">
-      		<mu1>1.1</mu1>
-      		<mu2>1.1</mu2>
-    	</gazebo>
 		<link name="${prefix}link_2">
 			<!--
@@ -74,5 +64,5 @@
 				<origin xyz="0.039 0 0.0075" rpy="0 0 0"/>
 				<geometry>
-                                        <mesh filename="package://robotiq_3f_gripper_visualization/meshes/robotiq-3f-gripper_articulated/visual/link_2.STL" />
+                                        <mesh filename="package://robotiq_3f_gripper_visualization/meshes/robotiq-3f-gripper_articulated/visual/link_2.dae" />
 				</geometry>
 				<material name="gray"/>
@@ -91,13 +81,9 @@
             </inertial>
 		</link>
-		<gazebo reference="${prefix}link_2">
-      		<mu1>1.1</mu1>
-      		<mu2>1.1</mu2>
-    	</gazebo>
 		<link name="${prefix}link_3">
 			<visual>
 				<origin xyz="0 0 0" rpy="0 0 0.52"/>
 				<geometry>
-                                        <mesh filename="package://robotiq_3f_gripper_visualization/meshes/robotiq-3f-gripper_articulated/visual/link_3.STL" />
+                                        <mesh filename="package://robotiq_3f_gripper_visualization/meshes/robotiq-3f-gripper_articulated/visual/link_3.dae" />
 				</geometry>
 				<material name="gray"/>
@@ -116,11 +102,9 @@
             </inertial>
 		</link>
-		<gazebo reference="${prefix}link_3">
-      		<mu1>1.1</mu1>
-      		<mu2>1.1</mu2>
-    	</gazebo>
 		<!-- end of link list -->
+		<!-- finger transmissions -->
+		<xacro:robotiq_transmission prefix="${prefix}"/>
+		<!-- end of finger transmissions -->
 		<!-- joint list -->
-		<xacro:robotiq_transmission prefix="${prefix}" />
 		<joint name="${prefix}joint_1" type="revolute">
 			<parent link="${prefix}link_0"/>
@@ -128,5 +112,5 @@
 			<axis xyz="0 0 1"/>
 			<origin xyz="0.020 0 0" rpy="0 0 0"/>
-                        <limit lower="0.0495" upper="1.2218" effort="${e1}" velocity="${s1}"/>
+			<limit lower="0.0495" upper="1.2218" effort="100" velocity="100"/>
 		</joint>
 		<joint name="${prefix}joint_2" type="revolute">
@@ -135,5 +119,5 @@
 			<axis xyz="0 0 1"/>
 			<origin xyz="0.050 -.028 0" rpy="0 0 -0.52"/>
-                        <limit lower="0.0" upper="1.5708" effort="${e1}" velocity="${s1}"/>
+			<limit lower="0.0" upper="1.5708" effort="100" velocity="100"/>
 		</joint>
 		<joint name="${prefix}joint_3" type="revolute">
@@ -142,5 +126,5 @@
 			<axis xyz="0 0 1"/>
 			<origin xyz="0.039 0 0" rpy="0 0 0"/>
-                        <limit lower="-1.2217" upper="-0.074532925" effort="${e1}" velocity="${s1}"/>
+			<limit lower="-1.2217" upper="-0.0523" effort="100" velocity="100"/>
 		</joint>
 		<!-- end of joint list -->

Commit message: Mimic 3f gripper joints

File: src/robotiq/robotiq_3f_gripper_visualization/cfg/robotiq-3f-gripper_articulated_macro.xacro (robot description, xacro)
@@ -51,4 +51,5 @@
 			<origin xyz="-0.0455 0.0214 -0.036" rpy="0 3.1416 -1.57"/>
 			<limit lower="-0.192" upper="0.1784" effort="100" velocity="100"/>
+			<mimic joint="${prefix}palm_finger_1_joint" type="revolute" multiplier="1" offset="0" />
 		</joint>
 		<joint name="${prefix}palm_finger_middle_joint" type="fixed">
@@ -74,13 +75,8 @@
 			</actuator>
 		</transmission>
-		<transmission name="${prefix}palm_finger_2_trans">
-			<type>transmission_interface/SimpleTransmission</type>
-			<joint name="${prefix}palm_finger_2_joint">
-				<hardwareInterface>hardware_interface/EffortJointInterface</hardwareInterface>
-			</joint>
-			<actuator name="${prefix}palm_finger_2_motor">
-				<mechanicalReduction>1</mechanicalReduction>
-			</actuator>
-			</transmission>
-		</xacro:macro>
+		<plugin filename="libroboticsgroup_gazebo_mimic_joint_plugin.so" name="${prefix}mimic_palm">
+                <joint>${prefix}palm_finger_1_joint</joint>
+                <mimicJoint>${prefix}palm_finger_2_joint</mimicJoint>
+                <multiplier>1.0</multiplier>
+            </plugin>
 </robot>

File: src/robotiq/robotiq_3f_gripper_visualization/cfg/robotiq-3f-gripper_finger_articulated_macro.xacro (robot description, xacro)
@@ -120,4 +120,5 @@
 			<origin xyz="0.050 -.028 0" rpy="0 0 -0.52"/>
 			<limit lower="0.0" upper="1.5708" effort="100" velocity="100"/>
+			<mimic joint="${prefix}joint_1" multiplier="1" offset="0" />
 		</joint>
 		<joint name="${prefix}joint_3" type="revolute">
@@ -127,4 +128,5 @@
 			<origin xyz="0.039 0 0" rpy="0 0 0"/>
 			<limit lower="-1.2217" upper="-0.0523" effort="100" velocity="100"/>
+			<mimic joint="${prefix}joint_1" multiplier="1" offset="0" />
 		</joint>
 		<!-- end of joint list -->

File: src/robotiq/robotiq_3f_gripper_visualization/cfg/robotiq.transmission.xacro (robot description, xacro)
@@ -11,22 +11,18 @@
       </actuator>
     </transmission>
-    <transmission name="${prefix}joint_2_trans">
-      <type>transmission_interface/SimpleTransmission</type>
-      <joint name="${prefix}joint_2">
-        <hardwareInterface>hardware_interface/EffortJointInterface</hardwareInterface>
-      </joint>
-      <actuator name="${prefix}joint_2_motor">
-        <mechanicalReduction>1</mechanicalReduction>
-      </actuator>
-    </transmission>
-    <transmission name="${prefix}joint_3_trans">
-      <type>transmission_interface/SimpleTransmission</type>
-      <joint name="${prefix}joint_3">
-        <hardwareInterface>hardware_interface/EffortJointInterface</hardwareInterface>
-      </joint>
-      <actuator name="${prefix}joint_3_motor">
-        <mechanicalReduction>1</mechanicalReduction>
-      </actuator>
-    </transmission>
+    <gazebo>
+             <!-- loading plugin: mimic joints works in gazebo now-->
+             <plugin filename="libroboticsgroup_gazebo_mimic_joint_plugin.so" name="${prefix}mimic_robotiq_140_4">
+                <joint>${prefix}joint_1</joint>
+                <mimicJoint>${prefix}joint_2</mimicJoint>
+                <multiplier>1.0</multiplier>
+            </plugin>
+            <plugin filename="libroboticsgroup_gazebo_mimic_joint_plugin.so" name="${prefix}mimic_robotiq_140_2">
+                <joint>${prefix}joint_1</joint>
+                <mimicJoint>${prefix}joint_3</mimicJoint>
+                <multiplier>1.0</multiplier>
+                <!--<offset>0.0</offset>-->
+            </plugin>
+        </gazebo>
   </xacro:macro>
 </robot>

Commit message: Finger 2  palm joint with mimic

File: src/robotiq/robotiq_3f_gripper_visualization/cfg/robotiq-3f-gripper_articulated_macro.xacro (robot description, xacro)
@@ -51,5 +51,5 @@
 			<origin xyz="-0.0455 0.0214 -0.036" rpy="0 3.1416 -1.57"/>
 			<limit lower="-0.192" upper="0.1784" effort="100" velocity="100"/>
-			<mimic joint="${prefix}palm_finger_1_joint" type="revolute" multiplier="1" offset="0" />
+			<mimic joint="${prefix}palm_finger_1_joint" type="revolute" multiplier="-1" offset="0" />
 		</joint>
 		<joint name="${prefix}palm_finger_middle_joint" type="fixed">
@@ -78,5 +78,6 @@
                 <joint>${prefix}palm_finger_1_joint</joint>
                 <mimicJoint>${prefix}palm_finger_2_joint</mimicJoint>
-                <multiplier>1.0</multiplier>
-            </plugin>
+                <multiplier>-1.0</multiplier>
+        </plugin>
+		</xacro:macro>
 </robot>

Commit message: Palm joint fixed

File: src/robotiq/robotiq_3f_gripper_visualization/cfg/robotiq-3f-gripper_articulated_macro.xacro (robot description, xacro)
@@ -38,5 +38,5 @@
 		<!-- end of link list -->
 		<!-- joint list -->
-		<joint name="${prefix}palm_finger_1_joint" type="revolute">
+		<joint name="${prefix}palm_finger_1_joint" type="fixed">
 			<parent link="${prefix}palm"/>
 			<child link="${prefix}finger_1_link_0"/>
@@ -45,5 +45,5 @@
 			<limit lower="-0.1784" upper="0.192" effort="100" velocity="100"/>
 		</joint>
-		<joint name="${prefix}palm_finger_2_joint" type="revolute">
+		<joint name="${prefix}palm_finger_2_joint" type="fixed">
 			<parent link="${prefix}palm"/>
 			<child link="${prefix}finger_2_link_0"/>
@@ -66,5 +66,5 @@
 		<!-- end of joint list -->
 		<!-- Palm transmissions -->
-		<transmission name="${prefix}palm_finger_1_trans">
+		<!--transmission name="${prefix}palm_finger_1_trans">
 			<type>transmission_interface/SimpleTransmission</type>
 			<joint name="${prefix}palm_finger_1_joint">
@@ -79,5 +79,5 @@
                 <mimicJoint>${prefix}palm_finger_2_joint</mimicJoint>
                 <multiplier>-1.0</multiplier>
-        </plugin>
+        </plugin-->
 		</xacro:macro>
 </robot>
