Commit message: Add transmissions to each 3f gripper finger

File: src/robotiq/robotiq_3f_gripper_visualization/cfg/robotiq.transmission.xacro (robot description, xacro)
@@ -11,18 +11,34 @@
       </actuator>
     </transmission>
-    <gazebo>
-             <!-- loading plugin: mimic joints works in gazebo now-->
-             <plugin filename="libroboticsgroup_gazebo_mimic_joint_plugin.so" name="${prefix}mimic_robotiq_140_4">
-                <joint>${prefix}joint_1</joint>
-                <mimicJoint>${prefix}joint_2</mimicJoint>
-                <multiplier>1.0</multiplier>
-            </plugin>
-            <plugin filename="libroboticsgroup_gazebo_mimic_joint_plugin.so" name="${prefix}mimic_robotiq_140_2">
-                <joint>${prefix}joint_1</joint>
-                <mimicJoint>${prefix}joint_3</mimicJoint>
-                <multiplier>1.0</multiplier>
-                <!--<offset>0.0</offset>-->
-            </plugin>
-        </gazebo>
+    <transmission name="${prefix}joint_2_trans">
+      <type>transmission_interface/SimpleTransmission</type>
+      <joint name="${prefix}joint_2">
+        <hardwareInterface>hardware_interface/EffortJointInterface</hardwareInterface>
+      </joint>
+      <actuator name="${prefix}joint_2_motor">
+        <mechanicalReduction>1</mechanicalReduction>
+      </actuator>
+    </transmission>
+    <transmission name="${prefix}joint_3_trans">
+      <type>transmission_interface/SimpleTransmission</type>
+      <joint name="${prefix}joint_3">
+        <hardwareInterface>hardware_interface/EffortJointInterface</hardwareInterface>
+      </joint>
+      <actuator name="${prefix}joint_3_motor">
+        <mechanicalReduction>1</mechanicalReduction>
+      </actuator>
+    </transmission>
+    <!-- <gazebo>
+      <plugin filename="libroboticsgroup_gazebo_mimic_joint_plugin.so" name="${prefix}mimic_robotiq_140_4">
+        <joint>${prefix}joint_1</joint>
+        <mimicJoint>${prefix}joint_2</mimicJoint>
+        <multiplier>1.0</multiplier>
+      </plugin>
+      <plugin filename="libroboticsgroup_gazebo_mimic_joint_plugin.so" name="${prefix}mimic_robotiq_140_2">
+        <joint>${prefix}joint_1</joint>
+        <mimicJoint>${prefix}joint_3</mimicJoint>
+        <multiplier>1.0</multiplier>
+      </plugin>
+    </gazebo> -->
   </xacro:macro>
 </robot>
