Commit message: Comment contact sensor plugin for 3f gripper

File: src/robotiq/robotiq_3f_gripper_visualization/cfg/robotiq-3f-gripper_finger_articulated_macro.xacro (robot description, xacro)
@@ -42,5 +42,5 @@
 				<material name="gray"/>
 			</visual>
-			<collision>
+			<collision name="${prefix}link_1_collision">
 				<origin xyz="0.050 -.028 0" rpy="0 0 -0.52"/>
 				<geometry>
@@ -68,5 +68,5 @@
 				<material name="gray"/>
 			</visual>
-			<collision>
+			<collision name="${prefix}link_2_collision">
 				<origin xyz="0.039 0 0.0075" rpy="0 0 0"/>
 				<geometry>
@@ -89,5 +89,5 @@
 				<material name="gray"/>
 			</visual>
-			<collision>
+			<collision name="${prefix}link_3_collision">
 				<origin xyz="0 0 0" rpy="0 0 0.52"/>
 				<geometry>
@@ -102,4 +102,58 @@
             </inertial>
 		</link>
+		<!-- <gazebo reference="${prefix}link_1">
+			<material>Gazebo/Grey</material>
+			<kp>100.0</kp>
+			<kd>10.0</kd>
+			<mu1>30.0</mu1>
+			<mu2>30.0</mu2>
+			<sensor type="contact" name="${prefix}link_1_contact_sensor">
+			<update_rate>30</update_rate>
+			<always_on>true</always_on>
+			<contact>
+				<collision>${prefix}link_1_collision_collision</collision>
+			</contact>
+			<plugin name="${prefix}link_1_plugin" filename="libgazebo_ros_bumper.so">
+				<bumperTopicName>${prefix}link_1_contact_sensor</bumperTopicName>
+				<frameName>${prefix}link_1</frameName>
+			</plugin>
+			</sensor>
+		</gazebo>
+		<gazebo reference="${prefix}link_2">
+			<material>Gazebo/Grey</material>
+			<kp>100.0</kp>
+			<kd>10.0</kd>
+			<mu1>30.0</mu1>
+			<mu2>30.0</mu2>
+			<sensor type="contact" name="${prefix}link_2_contact_sensor">
+			<update_rate>30</update_rate>
+			<always_on>true</always_on>
+			<contact>
+				<collision>${prefix}link_2_collision_collision</collision>
+			</contact>
+			<plugin name="${prefix}link_2_plugin" filename="libgazebo_ros_bumper.so">
+				<bumperTopicName>${prefix}link_2_contact_sensor</bumperTopicName>
+				<frameName>${prefix}link_2</frameName>
+			</plugin>
+			</sensor>
+		</gazebo>
+		<gazebo reference="${prefix}link_3">
+			<material>Gazebo/Grey</material>
+			<kp>100.0</kp>
+			<kd>10.0</kd>
+			<mu1>30.0</mu1>
+			<mu2>30.0</mu2>
+			<sensor type="contact" name="${prefix}link_3_contact_sensor">
+			<update_rate>30</update_rate>
+			<always_on>true</always_on>
+			<contact>
+				<collision>${prefix}link_3_collision_collision</collision>
+			</contact>
+			<plugin name="${prefix}link_3_plugin" filename="libgazebo_ros_bumper.so">
+				<bumperTopicName>${prefix}link_3_contact_sensor</bumperTopicName>
+				<frameName>${prefix}link_3</frameName>
+			</plugin>
+			</sensor>
+		</gazebo> -->
 		<!-- end of link list -->
 		<!-- finger transmissions -->
@@ -112,5 +166,5 @@
 			<axis xyz="0 0 1"/>
 			<origin xyz="0.020 0 0" rpy="0 0 0"/>
-			<limit lower="0.0495" upper="1.2218" effort="100" velocity="100"/>
+			<limit lower="0.0" upper="1.2218" effort="100" velocity="100"/>
 		</joint>
 		<joint name="${prefix}joint_2" type="revolute">
