Commit message: Increase velocity limits

File: src/universal_robot/ur_e_description/urdf/ur5e.urdf.xacro (robot description, xacro)
@@ -101,5 +101,5 @@
       <axis xyz="0 0 1" />
       <xacro:unless value="${joint_limited}">
-        <limit lower="${-2.0 * pi}" upper="${2.0 * pi}" effort="150.0" velocity="3.14"/>
+        <limit lower="${-2.0 * pi}" upper="${2.0 * pi}" effort="400.0" velocity="50"/>
         <xacro:if value="${safety_limits}">
           <safety_controller soft_lower_limit="${-2.0 * pi + safety_pos_margin}" soft_upper_limit="${2.0 * pi - safety_pos_margin}" k_position="${safety_k_position}" k_velocity="0.0"/>
@@ -138,5 +138,5 @@
       <axis xyz="0 1 0" />
       <xacro:unless value="${joint_limited}">
-        <limit lower="${-2.0 * pi}" upper="${2.0 * pi}" effort="150.0" velocity="3.14"/>
+        <limit lower="${-2.0 * pi}" upper="${2.0 * pi}" effort="400.0" velocity="50"/>
         <xacro:if value="${safety_limits}">
           <safety_controller soft_lower_limit="${-2.0 * pi + safety_pos_margin}" soft_upper_limit="${2.0 * pi - safety_pos_margin}" k_position="${safety_k_position}" k_velocity="0.0"/>
@@ -175,5 +175,5 @@
       <axis xyz="0 1 0" />
       <xacro:unless value="${joint_limited}">
-        <limit lower="${-pi}" upper="${pi}" effort="150.0" velocity="3.14"/>
+        <limit lower="${-pi}" upper="${pi}" effort="400.0" velocity="50"/>
         <xacro:if value="${safety_limits}">
           <safety_controller soft_lower_limit="${-2.0 * pi + safety_pos_margin}" soft_upper_limit="${2.0 * pi - safety_pos_margin}" k_position="${safety_k_position}" k_velocity="0.0"/>
@@ -212,5 +212,5 @@
       <axis xyz="0 1 0" />
       <xacro:unless value="${joint_limited}">
-        <limit lower="${-2.0 * pi}" upper="${2.0 * pi}" effort="28.0" velocity="6.28"/>
+        <limit lower="${-2.0 * pi}" upper="${2.0 * pi}" effort="50.0" velocity="12"/>
         <xacro:if value="${safety_limits}">
           <safety_controller soft_lower_limit="${-2.0 * pi + safety_pos_margin}" soft_upper_limit="${2.0 * pi - safety_pos_margin}" k_position="${safety_k_position}" k_velocity="0.0"/>
@@ -249,5 +249,5 @@
       <axis xyz="0 0 1" />
       <xacro:unless value="${joint_limited}">
-        <limit lower="${-2.0 * pi}" upper="${2.0 * pi}" effort="28.0" velocity="6.28"/>
+        <limit lower="${-2.0 * pi}" upper="${2.0 * pi}" effort="50.0" velocity="12"/>
         <xacro:if value="${safety_limits}">
           <safety_controller soft_lower_limit="${-2.0 * pi + safety_pos_margin}" soft_upper_limit="${2.0 * pi - safety_pos_margin}" k_position="${safety_k_position}" k_velocity="0.0"/>
@@ -286,5 +286,5 @@
       <axis xyz="0 1 0" />
       <xacro:unless value="${joint_limited}">
-        <limit lower="${-2.0 * pi}" upper="${2.0 * pi}" effort="28.0" velocity="6.28"/>
+        <limit lower="${-2.0 * pi}" upper="${2.0 * pi}" effort="50.0" velocity="12"/>
         <xacro:if value="${safety_limits}">
           <safety_controller soft_lower_limit="${-2.0 * pi + safety_pos_margin}" soft_upper_limit="${2.0 * pi - safety_pos_margin}" k_position="${safety_k_position}" k_velocity="0.0"/>

Commit message: Velocity and effort limits as parameters

File: src/universal_robot/ur_e_description/urdf/ur5e.urdf.xacro (robot description, xacro)
@@ -77,4 +77,8 @@
     <xacro:property name="forearm_radius" value="0.040" />    <!-- manually measured -->
     <xacro:property name="wrist_radius" value="0.045" />      <!-- manually measured -->
+    <xacro:property name="velocity_base" value="3.14" />
+    <xacro:property name="velocity_wrist" value="6.28" />
+    <xacro:property name="effort_base" value="150" />
+    <xacro:property name="effort_wrist" value="28" />
     <link name="${prefix}base_link" >
       <visual>
@@ -101,5 +105,5 @@
       <axis xyz="0 0 1" />
       <xacro:unless value="${joint_limited}">
-        <limit lower="${-2.0 * pi}" upper="${2.0 * pi}" effort="400.0" velocity="50"/>
+        <limit lower="${-2.0 * pi}" upper="${2.0 * pi}" effort="${effort_base}" velocity="${velocity_base}"/>
         <xacro:if value="${safety_limits}">
           <safety_controller soft_lower_limit="${-2.0 * pi + safety_pos_margin}" soft_upper_limit="${2.0 * pi - safety_pos_margin}" k_position="${safety_k_position}" k_velocity="0.0"/>
@@ -138,5 +142,5 @@
       <axis xyz="0 1 0" />
       <xacro:unless value="${joint_limited}">
-        <limit lower="${-2.0 * pi}" upper="${2.0 * pi}" effort="400.0" velocity="50"/>
+        <limit lower="${-2.0 * pi}" upper="${2.0 * pi}" effort="${effort_base}" velocity="${velocity_base}"/>
         <xacro:if value="${safety_limits}">
           <safety_controller soft_lower_limit="${-2.0 * pi + safety_pos_margin}" soft_upper_limit="${2.0 * pi - safety_pos_margin}" k_position="${safety_k_position}" k_velocity="0.0"/>
@@ -175,5 +179,5 @@
       <axis xyz="0 1 0" />
       <xacro:unless value="${joint_limited}">
-        <limit lower="${-pi}" upper="${pi}" effort="400.0" velocity="50"/>
+        <limit lower="${-pi}" upper="${pi}" effort="${effort_base}" velocity="${velocity_base}"/>
         <xacro:if value="${safety_limits}">
           <safety_controller soft_lower_limit="${-2.0 * pi + safety_pos_margin}" soft_upper_limit="${2.0 * pi - safety_pos_margin}" k_position="${safety_k_position}" k_velocity="0.0"/>
@@ -212,5 +216,5 @@
       <axis xyz="0 1 0" />
       <xacro:unless value="${joint_limited}">
-        <limit lower="${-2.0 * pi}" upper="${2.0 * pi}" effort="50.0" velocity="12"/>
+        <limit lower="${-2.0 * pi}" upper="${2.0 * pi}" effort="${effort_wrist}" velocity="${velocity_wrist}"/>
         <xacro:if value="${safety_limits}">
           <safety_controller soft_lower_limit="${-2.0 * pi + safety_pos_margin}" soft_upper_limit="${2.0 * pi - safety_pos_margin}" k_position="${safety_k_position}" k_velocity="0.0"/>
@@ -249,5 +253,5 @@
       <axis xyz="0 0 1" />
       <xacro:unless value="${joint_limited}">
-        <limit lower="${-2.0 * pi}" upper="${2.0 * pi}" effort="50.0" velocity="12"/>
+        <limit lower="${-2.0 * pi}" upper="${2.0 * pi}" effort="${effort_wrist}" velocity="${velocity_wrist}"/>
         <xacro:if value="${safety_limits}">
           <safety_controller soft_lower_limit="${-2.0 * pi + safety_pos_margin}" soft_upper_limit="${2.0 * pi - safety_pos_margin}" k_position="${safety_k_position}" k_velocity="0.0"/>
@@ -286,5 +290,5 @@
       <axis xyz="0 1 0" />
       <xacro:unless value="${joint_limited}">
-        <limit lower="${-2.0 * pi}" upper="${2.0 * pi}" effort="50.0" velocity="12"/>
+        <limit lower="${-2.0 * pi}" upper="${2.0 * pi}" effort="${effort_wrist}" velocity="${velocity_wrist}"/>
         <xacro:if value="${safety_limits}">
           <safety_controller soft_lower_limit="${-2.0 * pi + safety_pos_margin}" soft_upper_limit="${2.0 * pi - safety_pos_margin}" k_position="${safety_k_position}" k_velocity="0.0"/>

Commit message: Increase joint velocity

File: src/universal_robot/ur_e_description/urdf/ur5e.urdf.xacro (robot description, xacro)
@@ -77,6 +77,6 @@
     <xacro:property name="forearm_radius" value="0.040" />    <!-- manually measured -->
     <xacro:property name="wrist_radius" value="0.045" />      <!-- manually measured -->
-    <xacro:property name="velocity_base" value="3.14" />
-    <xacro:property name="velocity_wrist" value="6.28" />
+    <xacro:property name="velocity_base" value="8" /> <!-- 3.14 -->
+    <xacro:property name="velocity_wrist" value="10" /> <!-- 6.28 -->
     <xacro:property name="effort_base" value="150" />
     <xacro:property name="effort_wrist" value="28" />
@@ -354,5 +354,5 @@
       <child link="${prefix}tool0"/>
     </joint>
-    <gazebo reference="shoulder_pan_joint">
+    <!-- <gazebo reference="shoulder_pan_joint">
         <provideFeedback>true</provideFeedback>
     </gazebo>
@@ -413,5 +413,5 @@
             <jointName>wrist_3_joint</jointName>
         </plugin>
-    </gazebo>
+    </gazebo> -->
   </xacro:macro>
 </robot>
