Commit message: Delete URDF camera

File: src/universal_robot/ur_e_description/urdf/ur5e_robot.urdf.xacro (robot description, xacro)
@@ -6,14 +6,4 @@
   <xacro:include filename="$(find robotiq_2f_140_gripper_visualization)/urdf/robotiq_arg2f_140_model_macro.xacro" />
   <xacro:include filename="$(find robotiq_3f_gripper_visualization)/cfg/robotiq-3f-gripper_articulated_macro.xacro" />
-  <xacro:include filename="$(find ur_e_description)/urdf/camera/camera.urdf.xacro"/>
-  <xacro:include filename="$(find ur_e_description)/urdf/camera2/camera.urdf.xacro"/>
-  <xacro:camera_v0 parent="base_link">
-	     <origin xyz="1.5 0.0 0.5" rpy="0 0.0 3.1415"/>
-  </xacro:camera_v0>
-  <xacro:camera_gazebo_v0 />
-  <xacro:camera_v1 parent="base_link">
-	     <origin xyz="0.0 1.5 0.5" rpy="0 0.0 -1.57"/>
-  </xacro:camera_v1>
-  <xacro:camera_gazebo_v1 />
   <!-- ur5e -->
   <xacro:include filename="$(find ur_e_description)/urdf/ur5e.urdf.xacro" />

Commit message: Xacro file for the 2f gripper

File: src/universal_robot/ur_e_description/urdf/ur5e_robot.urdf.xacro (robot description, xacro)
@@ -5,5 +5,4 @@
   <xacro:include filename="$(find ur_e_description)/urdf/common.gazebo.xacro" />
   <xacro:include filename="$(find robotiq_2f_140_gripper_visualization)/urdf/robotiq_arg2f_140_model_macro.xacro" />
-  <xacro:include filename="$(find robotiq_3f_gripper_visualization)/cfg/robotiq-3f-gripper_articulated_macro.xacro" />
   <!-- ur5e -->
   <xacro:include filename="$(find ur_e_description)/urdf/ur5e.urdf.xacro" />
@@ -22,15 +21,3 @@
       <origin xyz=" 0.0 0.0 0.0" rpy="0.0 0.0 ${pi/2}" />
     </joint>
-    <link name="tool" />
-    <joint name="tool_tip" type="fixed">
-      <parent link= "ee_link" />
-      <child link = "tool" />
-      <origin xyz=" 0.00 0.0 0.2" rpy="0.0 0.0 0.0" />
-    </joint>
-  <!--xacro:robotiq-3f-gripper_articulated prefix="gripper_"/>
-    <joint name="base_gripper" type="fixed">
-      <parent link= "tool0" />
-      <child link = "gripper_palm" />
-      <origin xyz=" 0.0 0.0 0.1" rpy="${pi/2} 0.0 0.0" />
-    </joint-->
 </robot>

Commit message: Comments

File: src/universal_robot/ur_e_description/urdf/ur5e_robot.urdf.xacro (robot description, xacro)
@@ -1,12 +1,11 @@
 <?xml version="1.0"?>
-<robot xmlns:xacro="http://ros.org/wiki/xacro"
-       name="ur5e" >
+<robot xmlns:xacro="http://ros.org/wiki/xacro" name="ur5e" >
   <!-- common stuff -->
   <xacro:include filename="$(find ur_e_description)/urdf/common.gazebo.xacro" />
-  <xacro:include filename="$(find robotiq_2f_140_gripper_visualization)/urdf/robotiq_arg2f_140_model_macro.xacro" />
   <!-- ur5e -->
   <xacro:include filename="$(find ur_e_description)/urdf/ur5e.urdf.xacro" />
   <!-- arm -->
   <xacro:ur5e_robot prefix="" joint_limited="false"/>
+  <!-- world link and world joint-->
   <link name="world" />
   <joint name="world_joint" type="fixed">
@@ -15,9 +14,11 @@
     <origin xyz="0.0 0.0 0.0" rpy="0.0 0.0 0.0" />
   </joint>
- <xacro:robotiq_arg2f_140 prefix="" />
-    <joint name="ur5_ee_link_gripper_base" type="fixed">
-      <parent link= "tool0" />
-      <child link = "robotiq_arg2f_base_link" />
-      <origin xyz=" 0.0 0.0 0.0" rpy="0.0 0.0 ${pi/2}" />
-    </joint>
+  <!-- 2f gripper macro and robot / gripper fixed joint -->
+  <xacro:include filename="$(find robotiq_2f_140_gripper_visualization)/urdf/robotiq_arg2f_140_model_macro.xacro" />
+  <xacro:robotiq_arg2f_140 prefix="" />
+  <joint name="ur5_ee_link_gripper_base" type="fixed">
+    <parent link= "tool0" />
+    <child link = "robotiq_arg2f_base_link" />
+    <origin xyz=" 0.0 0.0 0.0" rpy="0.0 0.0 ${pi/2}" />
+  </joint>
 </robot>

File: src/universal_robot/ur_e_description/urdf/ur5e_robot_3f.urdf.xacro (robot description, xacro)
@@ -1,12 +1,11 @@
 <?xml version="1.0"?>
-<robot xmlns:xacro="http://ros.org/wiki/xacro"
-       name="ur5e" >
+<robot xmlns:xacro="http://ros.org/wiki/xacro" name="ur5e" >
   <!-- common stuff -->
   <xacro:include filename="$(find ur_e_description)/urdf/common.gazebo.xacro" />
-  <xacro:include filename="$(find robotiq_3f_gripper_visualization)/cfg/robotiq-3f-gripper_articulated_macro.xacro" />
   <!-- ur5e -->
   <xacro:include filename="$(find ur_e_description)/urdf/ur5e.urdf.xacro" />
   <!-- arm -->
   <xacro:ur5e_robot prefix="" joint_limited="false"/>
+  <!-- world link and world joint-->
   <link name="world" />
   <joint name="world_joint" type="fixed">
@@ -15,10 +14,10 @@
     <origin xyz="0.0 0.0 0.0" rpy="0.0 0.0 0.0" />
   </joint>
-  <xacro:robotiq-3f-gripper_articulated prefix="" parent="ee_link" reflect="1">
-    <origin rpy="0 0 ${-pi/2.0}" xyz="0.051 0 0"/>
-  </xacro:robotiq-3f-gripper_articulated>
+  <!-- 3f gripper macro and robot / gripper fixed joint -->
+  <xacro:include filename="$(find robotiq_3f_gripper_visualization)/cfg/robotiq-3f-gripper_articulated_macro.xacro" />
+  <xacro:robotiq-3f-gripper_articulated prefix="gripper_"/>
   <joint name="robotiq_hand_joint" type="fixed">
     <parent link="tool0"/>
-    <child link="palm"/>
+    <child link="gripper_palm"/>
     <origin xyz="0 0 0.02" rpy="1.57 0 0"/>
   </joint>

Commit message: Attach camera tool to robot end effector

File: src/universal_robot/ur_e_description/urdf/ur5e_robot.urdf.xacro (robot description, xacro)
@@ -3,4 +3,6 @@
   <!-- common stuff -->
   <xacro:include filename="$(find ur_e_description)/urdf/common.gazebo.xacro" />
+  <!-- Cameras -->
+  <xacro:include filename="$(find ur_e_description)/urdf/camera/camera.urdf.xacro"/>
   <!-- ur5e -->
   <xacro:include filename="$(find ur_e_description)/urdf/ur5e.urdf.xacro" />
@@ -22,3 +24,7 @@
     <origin xyz=" 0.0 0.0 0.0" rpy="0.0 0.0 ${pi/2}" />
   </joint>
+  <xacro:camera_v0 parent="tool0">
+	     <origin xyz="0.0 -0.1 0.02" rpy="0.0 -2 4.7226"/>
+  </xacro:camera_v0>
+  <xacro:camera_gazebo_v0 />
 </robot>

File: src/universal_robot/ur_e_description/urdf/ur5e_robot_3f.urdf.xacro (robot description, xacro)
@@ -3,4 +3,6 @@
   <!-- common stuff -->
   <xacro:include filename="$(find ur_e_description)/urdf/common.gazebo.xacro" />
+  <!-- Cameras -->
+  <xacro:include filename="$(find ur_e_description)/urdf/camera/camera.urdf.xacro"/>
   <!-- ur5e -->
   <xacro:include filename="$(find ur_e_description)/urdf/ur5e.urdf.xacro" />
@@ -22,3 +24,7 @@
     <origin xyz="0 0 0.02" rpy="1.57 0 0"/>
   </joint>
+  <xacro:camera_v0 parent="tool0">
+	     <origin xyz="0.0 -0.1 0.03" rpy="0.0 -1.9 4.7226"/>
+  </xacro:camera_v0>
+  <xacro:camera_gazebo_v0 />
 </robot>

Commit message: Add cameras to URDF robot files

File: src/universal_robot/ur_e_description/urdf/ur5e_robot.urdf.xacro (robot description, xacro)
@@ -24,7 +24,19 @@
     <origin xyz=" 0.0 0.0 0.0" rpy="0.0 0.0 ${pi/2}" />
   </joint>
-  <xacro:camera_v0 parent="tool0">
-	     <origin xyz="0.0 -0.1 0.02" rpy="0.0 -2 4.7226"/>
+  <!-- Camera joints -->
+  <!-- Tool Camera -->
+  <xacro:camera_v0 prefix="tool" parent="tool0">
+	     <origin xyz="0.0 -0.1 0.03" rpy="0.0 -1.9 4.7226"/>
   </xacro:camera_v0>
-  <xacro:camera_gazebo_v0 />
+  <xacro:camera_gazebo_v0 prefix="tool"/>
+  <!-- Y axis Camera-->
+  <xacro:camera_v0 prefix="y" parent="world">
+	     <origin xyz="0.5 0.6 0.17" rpy="0.0 0.0 4.712"/>
+  </xacro:camera_v0>
+  <xacro:camera_gazebo_v0 prefix="y"/>
+  <!-- X axis Camera-->
+  <xacro:camera_v0 prefix="x" parent="world">
+	     <origin xyz="1 0.0 0.17" rpy="0.0 0.0 3.14"/>
+  </xacro:camera_v0>
+  <xacro:camera_gazebo_v0 prefix="x"/>
 </robot>

File: src/universal_robot/ur_e_description/urdf/ur5e_robot_3f.urdf.xacro (robot description, xacro)
@@ -24,7 +24,19 @@
     <origin xyz="0 0 0.02" rpy="1.57 0 0"/>
   </joint>
-  <xacro:camera_v0 parent="tool0">
+  <!-- Camera joints -->
+  <!-- Tool Camera -->
+  <xacro:camera_v0 prefix="tool" parent="tool0">
 	     <origin xyz="0.0 -0.1 0.03" rpy="0.0 -1.9 4.7226"/>
   </xacro:camera_v0>
-  <xacro:camera_gazebo_v0 />
+  <xacro:camera_gazebo_v0 prefix="tool"/>
+  <!-- Y axis Camera-->
+  <xacro:camera_v0 prefix="y" parent="world">
+	     <origin xyz="0.5 0.6 0.17" rpy="0.0 0.0 4.712"/>
+  </xacro:camera_v0>
+  <xacro:camera_gazebo_v0 prefix="y"/>
+  <!-- X axis Camera-->
+  <xacro:camera_v0 prefix="x" parent="world">
+	     <origin xyz="1 0.0 0.17" rpy="0.0 0.0 3.14"/>
+  </xacro:camera_v0>
+  <xacro:camera_gazebo_v0 prefix="x"/>
 </robot>
