Commit message: Pybullet models

File: src/pybullet/pybullet_description/models/urdf/ur5e_2f.urdf (robot description, URDF)
Before this commit: robot ur5e, 24 links, 23 joints
Links:
- link base_link_inertia: geometry collision mesh filename=ur5/collision/base.stl; visual mesh filename=ur5/visual/base.dae
- link forearm_link: geometry collision mesh filename=ur5/collision/forearm.stl; visual mesh filename=ur5/visual/forearm.dae
- link shoulder_link: geometry collision mesh filename=ur5/collision/shoulder.stl; visual mesh filename=ur5/visual/shoulder.dae
- link upper_arm_link: geometry collision mesh filename=ur5/collision/upperarm.stl; visual mesh filename=ur5/visual/upperarm.dae
- link wrist_1_link: geometry collision mesh filename=ur5/collision/wrist1.stl; visual mesh filename=ur5/visual/wrist1.dae
- link wrist_2_link: geometry collision mesh filename=ur5/collision/wrist2.stl; visual mesh filename=ur5/visual/wrist2.dae
- link wrist_3_link: geometry collision mesh filename=ur5/collision/wrist3.stl; visual mesh filename=ur5/visual/wrist3.dae

File: src/pybullet/pybullet_description/models/urdf/ur5e_3f.urdf (robot description, URDF)
Before this commit: robot ur5e_robot, 25 links, 24 joints
Links:
- link base_link_inertia: geometry collision mesh filename=./ur5/collision/base.stl; visual mesh filename=./ur5/visual/base.dae
- link forearm_link: geometry collision mesh filename=./ur5/collision/forearm.stl; visual mesh filename=./ur5/visual/forearm.dae
- link shoulder_link: geometry collision mesh filename=./ur5/collision/shoulder.stl; visual mesh filename=./ur5/visual/shoulder.dae
- link upper_arm_link: geometry collision mesh filename=./ur5/collision/upperarm.stl; visual mesh filename=./ur5/visual/upperarm.dae
- link wrist_1_link: geometry collision mesh filename=./ur5/collision/wrist1.stl; visual mesh filename=./ur5/visual/wrist1.dae
- link wrist_2_link: geometry collision mesh filename=./ur5/collision/wrist2.stl; visual mesh filename=./ur5/visual/wrist2.dae
- link wrist_3_link: geometry collision mesh filename=./ur5/collision/wrist3.stl; visual mesh filename=./ur5/visual/wrist3.dae
