Commit message: Modifications for real launch

File: src/pybullet/pybullet_description/models/urdf/ur5e_3f.urdf (robot description, URDF)
Before this commit: robot ur5e_robot, 25 links, 24 joints
Joints:
- joint palm_finger_1_joint: limit lower=-0.1784 upper=0.192 effort=100 velocity=100 -> (none); type revolute -> fixed
- joint palm_finger_2_joint: limit lower=-0.192 upper=0.1784 effort=100 velocity=100 -> (none); type revolute -> fixed

File: src/universal_robot/ur_e_description/urdf/camera/camera.gazebo.xacro (robot description, xacro)
@@ -3,40 +3,40 @@
   <xacro:macro name="camera_gazebo_v0" params="prefix">
 	 <gazebo reference="${prefix}_camera_link">
-          <sensor type="camera" name="${prefix}_robot_camera">
-            <update_rate>30.0</update_rate>
-            <camera name="${prefix}_robot_camera">
-              <pose>0 0 0 0 0 0</pose>
-              <horizontal_fov>1.3962634</horizontal_fov>
-              <image>
-                <width>640</width>
-                <height>480</height>
-                <format>R8G8B8</format>
-              </image>
-              <clip>
-               <near>0.02</near>
-               <far>300</far>
-              </clip>
-              <noise>
-                <type>gaussian</type>
-                <mean>0.0</mean>
-                <stddev>0.007</stddev>
-              </noise>
-            </camera>
-            <plugin name="camera_controller" filename="libgazebo_ros_camera.so">
-              <alwaysOn>true</alwaysOn>
-              <updateRate>0.0</updateRate>
-              <cameraName>${prefix}_robot_camera</cameraName>
-              <imageTopicName>image_raw</imageTopicName>
-              <cameraInfoTopicName>camera_info</cameraInfoTopicName>
-              <frameName>${prefix}_camera_link</frameName>
-              <hackBaseline>0.0</hackBaseline>
-              <distortionK1>0.0</distortionK1>
-              <distortionK2>0.0</distortionK2>
-              <distortionK3>0.0</distortionK3>
-              <distortionT1>0.0</distortionT1>
-              <distortionT2>0.0</distortionT2>
-            </plugin>
-          </sensor>
-        </gazebo>
+    <sensor type="camera" name="${prefix}_robot_camera">
+      <update_rate>30.0</update_rate>
+      <camera name="${prefix}_robot_camera">
+        <pose>0 0 0 0 0 0</pose>
+        <horizontal_fov>1.3962634</horizontal_fov>
+        <image>
+          <width>640</width>
+          <height>480</height>
+          <format>R8G8B8</format>
+        </image>
+        <clip>
+          <near>0.02</near>
+          <far>300</far>
+        </clip>
+        <noise>
+          <type>gaussian</type>
+          <mean>0.0</mean>
+          <stddev>0.007</stddev>
+        </noise>
+      </camera>
+      <plugin name="camera_controller" filename="libgazebo_ros_camera.so">
+        <alwaysOn>true</alwaysOn>
+        <updateRate>0.0</updateRate>
+        <cameraName>${prefix}_robot_camera</cameraName>
+        <imageTopicName>image_raw</imageTopicName>
+        <cameraInfoTopicName>camera_info</cameraInfoTopicName>
+        <frameName>${prefix}_camera_link</frameName>
+        <hackBaseline>0.0</hackBaseline>
+        <distortionK1>0.0</distortionK1>
+        <distortionK2>0.0</distortionK2>
+        <distortionK3>0.0</distortionK3>
+        <distortionT1>0.0</distortionT1>
+        <distortionT2>0.0</distortionT2>
+      </plugin>
+    </sensor>
+   </gazebo>
   </xacro:macro>
 </robot>

File: src/universal_robot/ur_e_description/urdf/ur5e_robot.urdf.xacro (robot description, xacro)
@@ -35,8 +35,3 @@
   </xacro:camera_v0>
   <xacro:camera_gazebo_v0 prefix="y"/>
-  <!-- X axis Camera-->
-  <xacro:camera_v0 prefix="x" parent="world">
-	     <origin xyz="1 0.0 0.17" rpy="0.0 0.0 3.14"/>
-  </xacro:camera_v0>
-  <xacro:camera_gazebo_v0 prefix="x"/>
 </robot>

File: src/universal_robot/ur_e_description/urdf/ur5e_robot_3f.urdf.xacro (robot description, xacro)
@@ -22,5 +22,5 @@
     <parent link="tool0"/>
     <child link="gripper_palm"/>
-    <origin xyz="0 0 0.02" rpy="1.57 0 0"/>
+    <origin xyz="0 0 0.03" rpy="1.57 0 0"/>
   </joint>
   <!-- Camera joints -->
@@ -35,8 +35,3 @@
   </xacro:camera_v0>
   <xacro:camera_gazebo_v0 prefix="y"/>
-  <!-- X axis Camera-->
-  <xacro:camera_v0 prefix="x" parent="world">
-	     <origin xyz="1 0.0 0.17" rpy="0.0 0.0 3.14"/>
-  </xacro:camera_v0>
-  <xacro:camera_gazebo_v0 prefix="x"/>
 </robot>
