Commit message: Add zero inertia to dummy links

File: src/objects_models/urdf/002_master_chef_can/model.urdf (robot description, URDF)
Before this commit: robot model.urdf, 2 links, 1 joints
Links:
- link dummy: mass None -> 0.01

File: src/objects_models/urdf/003_cracker_box/model.urdf (robot description, URDF)
Before this commit: robot model.urdf, 2 links, 1 joints
Links:
- link dummy: mass None -> 0.01

File: src/objects_models/urdf/004_sugar_box/model.urdf (robot description, URDF)
Before this commit: robot model.urdf, 2 links, 1 joints
Links:
- link dummy: mass None -> 0.01

File: src/objects_models/urdf/005_tomato_soup_can/model.urdf (robot description, URDF)
Before this commit: robot model.urdf, 2 links, 1 joints
Links:
- link dummy: mass None -> 0.01

File: src/objects_models/urdf/006_mustard_bottle/model.urdf (robot description, URDF)
Before this commit: robot model.urdf, 2 links, 1 joints
Links:
- link dummy: mass None -> 0.01

File: src/objects_models/urdf/007_tuna_fish_can/model.urdf (robot description, URDF)
Before this commit: robot tuna_fish_can, 2 links, 1 joints
Links:
- link dummy: mass None -> 0.01

File: src/objects_models/urdf/008_pudding_box/model.urdf (robot description, URDF)
Before this commit: robot model.urdf, 2 links, 1 joints
Links:
- link dummy: mass None -> 0.01

File: src/objects_models/urdf/009_gelatin_box/model.urdf (robot description, URDF)
Before this commit: robot model.urdf, 2 links, 1 joints
Links:
- link dummy: mass None -> 0.01

File: src/objects_models/urdf/010_potted_meat_can/model.urdf (robot description, URDF)
Before this commit: robot model.urdf, 2 links, 1 joints
Links:
- link dummy: mass None -> 0.01

File: src/objects_models/urdf/011_banana/model.urdf (robot description, URDF)
Before this commit: robot model.urdf, 2 links, 1 joints
Links:
- link dummy: mass None -> 0.01

File: src/objects_models/urdf/012_strawberry/model.urdf (robot description, URDF)
Before this commit: robot model.urdf, 2 links, 1 joints
Links:
- link dummy: mass None -> 0.01

File: src/objects_models/urdf/013_apple/model.urdf (robot description, URDF)
Before this commit: robot model.urdf, 2 links, 1 joints
Links:
- link baseLink: geometry collision mesh filename=package://objects_models/urdf/013_apple/collision.obj scale=1 1 1; visual mesh filename=package://objects_models/urdf/013_apple/textured.obj scale=1 1 1
- link dummy: mass None -> 0.01

File: src/objects_models/urdf/014_lemon/model.urdf (robot description, URDF)
Before this commit: robot model.urdf, 2 links, 1 joints
Links:
- link dummy: mass None -> 0.01

File: src/objects_models/urdf/015_peach/model.urdf (robot description, URDF)
Before this commit: robot model.urdf, 2 links, 1 joints
Links:
- link dummy: mass None -> 0.01

File: src/objects_models/urdf/016_pear/model.urdf (robot description, URDF)
Before this commit: robot model.urdf, 2 links, 1 joints
Links:
- link dummy: mass None -> 0.01

File: src/objects_models/urdf/017_orange/model.urdf (robot description, URDF)
Before this commit: robot model.urdf, 2 links, 1 joints
Links:
- link dummy: mass None -> 0.01

File: src/objects_models/urdf/018_plum/model.urdf (robot description, URDF)
Before this commit: robot model.urdf, 2 links, 1 joints
Links:
- link dummy: mass None -> 0.01

File: src/objects_models/urdf/021_bleach_cleanser/model.urdf (robot description, URDF)
Before this commit: robot model.urdf, 2 links, 1 joints
Links:
- link dummy: mass None -> 0.01

File: src/pybullet/pybullet_description/models/urdf/ur5e_3f.urdf (robot description, URDF)
Before this commit: robot ur5e_robot, 25 links, 24 joints
Links:
- link base: mass None -> 0
- link base_link: mass None -> 0
- link flange: mass None -> 0
- link palm: mass None -> 0
- link tool0: mass None -> 0
- link tool_grip: mass None -> 1.3
