Commit message: Add prefix to URDF parameters

File: src/universal_robot/ur_e_description/urdf/camera/camera.gazebo.xacro (robot description, xacro)
@@ -1,9 +1,9 @@
 <?xml version="1.0"?>
 <robot xmlns:xacro="http://ros.org/wiki/xacro">
-  <xacro:macro name="camera_gazebo_v0">
-	 <gazebo reference="camera_link">
-          <sensor type="camera" name="robot_camera2">
+  <xacro:macro name="camera_gazebo_v0" params="prefix">
+	 <gazebo reference="${prefix}_camera_link">
+          <sensor type="camera" name="${prefix}_robot_camera">
             <update_rate>30.0</update_rate>
-            <camera name="robot_camera">
+            <camera name="${prefix}_robot_camera">
               <pose>0 0 0 0 0 0</pose>
               <horizontal_fov>1.3962634</horizontal_fov>
@@ -26,8 +26,8 @@
               <alwaysOn>true</alwaysOn>
               <updateRate>0.0</updateRate>
-              <cameraName>robot_camera</cameraName>
+              <cameraName>${prefix}_robot_camera</cameraName>
               <imageTopicName>image_raw</imageTopicName>
               <cameraInfoTopicName>camera_info</cameraInfoTopicName>
-              <frameName>camera_link</frameName>
+              <frameName>${prefix}_camera_link</frameName>
               <hackBaseline>0.0</hackBaseline>
               <distortionK1>0.0</distortionK1>

File: src/universal_robot/ur_e_description/urdf/camera/camera.urdf.xacro (robot description, xacro)
@@ -2,12 +2,12 @@
 <robot name="delirobo" xmlns:xacro="http://ros.org/wiki/xacro">
   <xacro:include filename="$(find ur_e_description)/urdf/camera/camera.gazebo.xacro"/>
-  <xacro:macro name="camera_v0" params="parent *joint_origin">
-	<joint name="camera_joint" type="fixed">
+  <xacro:macro name="camera_v0" params="parent prefix *joint_origin">
+	<joint name="${prefix}_camera_joint" type="fixed">
 	  <xacro:insert_block name="joint_origin"/>
 	  <parent link="${parent}"/>
-	  <child link="camera_link"/>
+	  <child link="${prefix}_camera_link"/>
 	  <origin xyz="0.0 0.1 0.0" rpy="0.0 0.0 0.0" />
 	</joint>
-	<link name="camera_link">
+	<link name="${prefix}_camera_link">
 	  <visual>
 		<geometry>
